File: Hardware/PMK_Keyboard/PMK_Keyboard.kicad_pcb (KiCad board)
At the start: 2 copper layers, 61 parts, among them IC1 SN74HC165PWR, IC2 SN74HC165PWR, IC3 SN74HC165PWR, IC4 SN74HC165PWR, IC5 SN74HC165PWR, IC6 SN74HC165PWR, IC7 ESP32-S2FH4, SW1 SW_Push, SW10 SW_Push, SW11 SW_Push, SW12 SW_Push, SW13 SW_Push, SW14 SW_Push, SW15 SW_Push, SW16 SW_Push, SW17 SW_Push, SW18 SW_Push, SW19 SW_Push, SW2 SW_Push, SW20 SW_Push, SW21 SW_Push, SW22 SW_Push, SW23 SW_Push, SW24 SW_Push, SW25 SW_Push, SW26 SW_Push, SW27 SW_Push, SW28 SW_Push, SW29 SW_Push, SW3 SW_Push, SW30 SW_Push, SW31 SW_Push, SW32 SW_Push, SW33 SW_Push, SW34 SW_Push, SW35 SW_Push, SW36 SW_Push, SW37 SW_Push, SW38 SW_Push, SW39 SW_Push, SW4 SW_Push, SW40 SW_Push, SW41 SW_Push, SW42 SW_Push, SW43 SW_Push, SW44 SW_Push, SW45 SW_Push, SW46 SW_Push, SW47 SW_Push, SW48 SW_Push, SW5 SW_Push, SW6 SW_Push, SW7 SW_Push, SW8 SW_Push, SW9 SW_Push

Commit message: Added some sort of layout
Parts:
- added G***: LOGO, Component_lib:pmk-v1, F.Cu at (106.5, 101.7)
- moved IC1 198.6 mm to (-148.6, 23.0)
- moved IC2 198.6 mm to (-128.6, 23.0)
- moved IC3 198.6 mm to (-108.6, 23.0)
- moved IC4 198.6 mm to (-89.5, 23.2)
- moved IC5 198.6 mm to (-68.6, 23.0)
- moved IC6 198.6 mm to (-49.5, 23.0)
- moved IC7 198.6 mm to (-168.6, 18.0)
- moved RN1 198.6 mm to (-158.6, 23.0)
- moved RN2 198.6 mm to (-138.6, 23.0)
- moved RN3 198.6 mm to (-118.6, 23.0)
- moved RN4 198.6 mm to (-98.6, 23.0)
- moved RN5 198.6 mm to (-78.6, 23.0)
- moved RN6 198.6 mm to (-58.6, 23.0)
- moved SW1 198.6 mm to (-153.6, 38.0)
- moved SW10 198.6 mm to (-133.6, 56.8)
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
Commit message: firstlayouttest
Parts:
- moved SW16 250.3 mm to (81.2, 49.5)
- moved SW15 233.8 mm to (80.3, 63.7)
- moved SW8 231.4 mm to (67.5, 109.6)
- moved SW40 225.1 mm to (150.2, 153.4), turned to -30 degrees
- moved SW14 223.0 mm to (81.0, 77.4)
- moved SW7 222.9 mm to (66.8, 124.4)
- moved SW47 220.0 mm to (164.4, 128.7), turned to -30 degrees
- moved SW13 216.4 mm to (81.2, 91.9)
- moved SW39 215.6 mm to (141.3, 140.1), turned to -30 degrees
- moved SW48 214.1 mm to (157.3, 141.1), turned to -30 degrees
- moved SW19 208.9 mm to (95.3, 75.8)
- moved SW20 208.8 mm to (95.1, 90.4)
- moved SW17 208.7 mm to (94.9, 47.1)
- moved SW18 208.4 mm to (94.7, 61.6)
- moved SW46 206.3 mm to (152.1, 121.6), turned to -30 degrees
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
Commit message: trying some layout scale
Parts:
- moved G*** 140.4 mm to (242.0, 65.0)
- moved SW41 139.6 mm to (277.0, 38.0)
- moved SW42 139.5 mm to (277.0, 53.5)
- moved SW43 139.4 mm to (277.0, 69.0)
- moved SW44 139.3 mm to (277.0, 84.5)
- moved SW45 139.2 mm to (277.0, 100.0)
- moved SW33 138.3 mm to (261.5, 38.0)
- moved SW34 138.2 mm to (261.5, 53.5)
- moved SW35 138.1 mm to (261.5, 69.0)
- moved SW36 138.0 mm to (261.5, 84.5)
- moved SW37 137.9 mm to (261.5, 100.0)
- moved SW38 31.5 mm to (118.0, 162.5)
- moved SW39 31.5 mm to (130.3, 169.6)
- moved SW46 31.5 mm to (141.1, 151.1)
- moved SW47 31.5 mm to (153.4, 158.2)
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
Commit message: updated layout
Parts:
- moved G*** 149.6 mm to (103.8, 122.2)
- moved SW41 141.0 mm to (138.5, 64.2)
- moved SW42 140.9 mm to (138.5, 79.5)
- moved SW43 140.9 mm to (138.5, 94.8)
- moved SW44 140.8 mm to (138.5, 110.0)
- moved SW45 140.8 mm to (138.5, 125.2)
- moved SW33 140.7 mm to (123.2, 64.2)
- moved SW34 140.7 mm to (123.2, 79.5)
- moved SW35 140.6 mm to (123.2, 94.8)
- moved SW36 140.6 mm to (123.2, 110.0)
- moved SW37 140.5 mm to (123.2, 125.2)
- moved SW12 20.8 mm to (61.5, 112.2)
- moved SW22 20.5 mm to (77.0, 139.2)
- moved SW8 20.1 mm to (61.5, 127.5)
- moved SW6 20.0 mm to (46.0, 143.0)
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Other:
- board outline added: 152 x 134.8 mm
