File: Hardware/PMK_Keyboard/PMK_Keyboard.kicad_pcb (KiCad board)
At the start: 2 copper layers, 181.6 x 154.3 mm, 84 parts, among them IC1 SN74HC165PWR, IC2 SN74HC165PWR, IC3 SN74HC165PWR, IC4 SN74HC165PWR, IC5 SN74HC165PWR, IC7 ESP32-S2FH4, SW1 SW_Push, SW10 SW_Push, SW11 SW_Push, SW12 SW_Push, SW13 SW_Push, SW14 SW_Push, SW15 SW_Push, SW16 SW_Push, SW17 SW_Push, SW18 SW_Push, SW19 SW_Push, SW2 SW_Push, SW20 SW_Push, SW21 SW_Push, SW22 SW_Push, SW23 SW_Push, SW24 SW_Push, SW25 SW_Push, SW26 SW_Push, SW27 SW_Push, SW28 SW_Push, SW29 SW_Push, SW3 SW_Push, SW30 SW_Push, SW31 SW_Push, SW32 SW_Push, SW33 SW_Push, SW34 SW_Push, SW35 SW_Push, SW36 SW_Push, SW37 SW_Push, SW38 SW_Push, SW39 SW_Push, SW4 SW_Push, SW40 SW_Push, SW5 SW_Push, SW6 SW_Push, SW7 SW_Push, SW8 SW_Push, SW9 SW_Push, U1 MIC5528-3.3YMT-T5, Y1 40MHz

Commit message: Added LEDs
Parts:
- added C19: 10u, Capacitor_SMD:C_0603_1608Metric, F.Cu at (158.4, 29.8)
- added C20: 10u, Capacitor_SMD:C_0603_1608Metric, F.Cu at (158.4, 32.3)
- added D10: YF923_2020_WS2812_LED, Component_lib:YF923_2020_WS2812_LED_DUALSIDE, F.Cu at (58.5, 73.8)
- added D11: YF923_2020_WS2812_LED, Component_lib:YF923_2020_WS2812_LED_DUALSIDE, F.Cu at (77.5, 68.8)
- added D12: YF923_2020_WS2812_LED, Component_lib:YF923_2020_WS2812_LED_DUALSIDE, F.Cu at (96.5, 66.2)
- added D13: YF923_2020_WS2812_LED, Component_lib:YF923_2020_WS2812_LED_DUALSIDE, F.Cu at (116.0, 68.8)
- added D14: YF923_2020_WS2812_LED, Component_lib:YF923_2020_WS2812_LED_DUALSIDE, F.Cu at (135.0, 71.2)
- added D15: YF923_2020_WS2812_LED, Component_lib:YF923_2020_WS2812_LED_DUALSIDE, F.Cu at (154.0, 71.2)
- added D16: YF923_2020_WS2812_LED, Component_lib:YF923_2020_WS2812_LED_DUALSIDE, F.Cu at (154.0, 90.2)
- added D17: YF923_2020_WS2812_LED, Component_lib:YF923_2020_WS2812_LED_DUALSIDE, F.Cu at (135.0, 90.2)
- added D18: YF923_2020_WS2812_LED, Component_lib:YF923_2020_WS2812_LED_DUALSIDE, F.Cu at (116.0, 87.8)
- added D19: YF923_2020_WS2812_LED, Component_lib:YF923_2020_WS2812_LED_DUALSIDE, F.Cu at (96.5, 85.2)
- added D2: YF923_2020_WS2812_LED, Component_lib:YF923_2020_WS2812_LED_DUALSIDE, F.Cu at (154.0, 52.2)
- added D20: YF923_2020_WS2812_LED, Component_lib:YF923_2020_WS2812_LED_DUALSIDE, F.Cu at (77.5, 87.8)
- added D21: YF923_2020_WS2812_LED, Component_lib:YF923_2020_WS2812_LED_DUALSIDE, F.Cu at (58.5, 92.8)
- added D22: YF923_2020_WS2812_LED, Component_lib:YF923_2020_WS2812_LED_DUALSIDE, F.Cu at (35.0, 92.8)
- added D23: YF923_2020_WS2812_LED, Component_lib:YF923_2020_WS2812_LED_DUALSIDE, F.Cu at (35.0, 111.8)
- added D24: YF923_2020_WS2812_LED, Component_lib:YF923_2020_WS2812_LED_DUALSIDE, F.Cu at (58.5, 111.8)
- added D25: YF923_2020_WS2812_LED, Component_lib:YF923_2020_WS2812_LED_DUALSIDE, F.Cu at (77.5, 106.8)
- added D26: YF923_2020_WS2812_LED, Component_lib:YF923_2020_WS2812_LED_DUALSIDE, F.Cu at (96.5, 104.2)
- added D27: YF923_2020_WS2812_LED, Component_lib:YF923_2020_WS2812_LED_DUALSIDE, F.Cu at (116.0, 106.8)
- added D28: YF923_2020_WS2812_LED, Component_lib:YF923_2020_WS2812_LED_DUALSIDE, F.Cu at (135.0, 109.2)
- added D29: YF923_2020_WS2812_LED, Component_lib:YF923_2020_WS2812_LED_DUALSIDE, F.Cu at (154.0, 109.2)
- added D3: YF923_2020_WS2812_LED, Component_lib:YF923_2020_WS2812_LED_DUALSIDE, F.Cu at (135.0, 52.2)
- added D30: YF923_2020_WS2812_LED, Component_lib:YF923_2020_WS2812_LED_DUALSIDE, F.Cu at (170.1, 126.2)
- added D31: YF923_2020_WS2812_LED, Component_lib:YF923_2020_WS2812_LED_DUALSIDE, F.Cu at (186.9, 135.9)
- added D32: YF923_2020_WS2812_LED, Component_lib:YF923_2020_WS2812_LED_DUALSIDE, F.Cu at (177.3, 152.5)
- added D33: YF923_2020_WS2812_LED, Component_lib:YF923_2020_WS2812_LED_DUALSIDE, F.Cu at (167.7, 169.1)
- added D34: YF923_2020_WS2812_LED, Component_lib:YF923_2020_WS2812_LED_DUALSIDE, F.Cu at (156.1, 150.9)
- added D35: YF923_2020_WS2812_LED, Component_lib:YF923_2020_WS2812_LED_DUALSIDE, F.Cu at (139.2, 141.1)
- added D36: YF923_2020_WS2812_LED, Component_lib:YF923_2020_WS2812_LED_DUALSIDE, F.Cu at (116.0, 125.8)
- added D37: YF923_2020_WS2812_LED, Component_lib:YF923_2020_WS2812_LED_DUALSIDE, F.Cu at (96.5, 123.2)
- added D38: YF923_2020_WS2812_LED, Component_lib:YF923_2020_WS2812_LED_DUALSIDE, F.Cu at (77.5, 125.8)
- added D39: YF923_2020_WS2812_LED, Component_lib:YF923_2020_WS2812_LED_DUALSIDE, F.Cu at (58.5, 130.8)
- added D4: YF923_2020_WS2812_LED, Component_lib:YF923_2020_WS2812_LED_DUALSIDE, F.Cu at (116.0, 49.8)
- added D40: YF923_2020_WS2812_LED, Component_lib:YF923_2020_WS2812_LED_DUALSIDE, F.Cu at (40.0, 130.8)
- added D41: YF923_2020_WS2812_LED, Component_lib:YF923_2020_WS2812_LED_DUALSIDE, F.Cu at (27.5, 32.2)
- added D5: YF923_2020_WS2812_LED, Component_lib:YF923_2020_WS2812_LED_DUALSIDE, F.Cu at (96.5, 47.2)
- added D6: YF923_2020_WS2812_LED, Component_lib:YF923_2020_WS2812_LED_DUALSIDE, F.Cu at (77.5, 49.8)
- added D7: YF923_2020_WS2812_LED, Component_lib:YF923_2020_WS2812_LED_DUALSIDE, F.Cu at (58.5, 54.8)
- added D8: YF923_2020_WS2812_LED, Component_lib:YF923_2020_WS2812_LED_DUALSIDE, F.Cu at (35.0, 54.8)
- added D9: YF923_2020_WS2812_LED, Component_lib:YF923_2020_WS2812_LED_DUALSIDE, F.Cu at (35.0, 73.8)
- added U2: MIC5528-3.3YMT-T5, Component_lib:SON40P120X120X60-7N-D, F.Cu at (162.2, 30.2)
- moved U1 34.3 mm to (173.5, 28.2)
Connections:
- IC1 pad 1: /PL -> /IO36
- IC1 pad 2: /SPI_CLK -> /IO38
- IC1 pad 9: /SPI_MISO -> /IO37
- IC2 pad 1: /PL -> /IO36
- IC2 pad 2: /SPI_CLK -> /IO38
- IC3 pad 1: /PL -> /IO36
- IC3 pad 2: /SPI_CLK -> /IO38
- IC4 pad 1: /PL -> /IO36
- IC4 pad 2: /SPI_CLK -> /IO38
- IC5 pad 1: /PL -> /IO36
- IC5 pad 2: /SPI_CLK -> /IO38
- IC7 pad 39: /IO35 -> /CE
Routing:
- net VDD: track 0.00 -> 1176.4 mm, vias 0 -> 54
- net /SPI_CLK: track 149.3 -> 0.00 mm, vias 5 -> 0
- net /IO38: track 0.00 -> 149.3 mm, vias 0 -> 5
- net /PL: track 131.8 -> 0.00 mm, vias 5 -> 0
- net /IO36: track 0.00 -> 131.8 mm, vias 0 -> 5
- net GND: track 3.32 -> 102.8 mm, vias 0 -> 85
- net Net-(D35-Pad4): track 0.00 -> 32.5 mm, vias 0 -> 2
- net Net-(D29-Pad4): track 0.00 -> 28.9 mm, vias 0 -> 3
- net Net-(D32-Pad4): track 0.00 -> 28.3 mm, vias 0 -> 3
- net Net-(D31-Pad4): track 0.00 -> 28.0 mm, vias 0 -> 4
- net Net-(D33-Pad4): track 0.00 -> 26.6 mm, vias 0 -> 2
- net Net-(D21-Pad4): track 0.00 -> 26.4 mm, vias 0 -> 4
- net Net-(D10-Pad3): track 0.00 -> 26.4 mm, vias 0 -> 4
- net Net-(D23-Pad4): track 0.00 -> 25.6 mm, vias 0 -> 2
- net Net-(D7-Pad4): track 0.00 -> 25.5 mm, vias 0 -> 2
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- added copper zone on B.Cu, net GND

Commit message: added hierachic pages
Parts:
- turned IC7 to -90 degrees
