File: Hardware/PMK_Keyboard/PMK_Keyboard.kicad_sch (KiCad schematic)
At the start: 127 parts, among them IC1 SN74HC165PWR, IC2 SN74HC165PWR, IC3 SN74HC165PWR, IC4 SN74HC165PWR, IC5 SN74HC165PWR, IC7 ESP32-S2FH4, J10 USB_C_Receptacle_USB2.0, SW1 SW_Push, SW10 SW_Push, SW11 SW_Push, SW12 SW_Push, SW13 SW_Push, SW14 SW_Push, SW15 SW_Push, SW16 SW_Push, SW17 SW_Push, SW18 SW_Push, SW19 SW_Push, SW2 SW_Push, SW20 SW_Push, SW21 SW_Push, SW22 SW_Push, SW23 SW_Push, SW24 SW_Push, SW25 SW_Push, SW26 SW_Push, SW27 SW_Push, SW28 SW_Push, SW29 SW_Push, SW3 SW_Push, SW30 SW_Push, SW31 SW_Push, SW32 SW_Push, SW33 SW_Push, SW34 SW_Push, SW35 SW_Push, SW36 SW_Push, SW37 SW_Push, SW38 SW_Push, SW39 SW_Push, SW4 SW_Push, SW40 SW_Push, SW5 SW_Push, SW6 SW_Push, SW7 SW_Push, SW8 SW_Push, SW9 SW_Push, U1 MIC5528-3.3YMT-T5, U2 MIC5528-3.3YMT-T5, Y1 40MHz

Commit message: added hierachic pages
Parts:
- removed ANT1: 2450AT18A100E, Component_lib:ANTC3216X140N, symbol Component lib:2450AT18A100E
- removed C1, C19, C2, C20, C4: 10u, Capacitor_SMD:C_0603_1608Metric, symbol Component lib:C
- removed C10, C11: 15p, Capacitor_SMD:C_0201_0603Metric, symbol Component lib:C
- removed C12, C13, C14, C16, C3, C5, C7, C8, C9: 100n, Capacitor_SMD:C_0402_1005Metric, symbol Component lib:C
- removed C15, C6: 1u, Capacitor_SMD:C_0402_1005Metric, symbol Component lib:C
- removed C17, C18: C, Capacitor_SMD:C_0201_0603Metric, symbol Component lib:C
- removed D1: LED, LED_SMD:LED_0402_1005Metric, symbol Component lib:LED
- removed D10, D11, D12, D13, D14, D15, D16, D17, D18, D19, D2, D20, D21, D22, D23, D24, D25, D26, D27, D28, D29, D3, D30, D31, D32, D33, D34, D35, D36, D37, D38, D39, D4, D40, D41, D5, D6, D7, D8, D9: YF923_2020_WS2812_LED, Component_lib:YF923_2020_WS2812_LED_DUALSIDE, symbol Component lib:YF923_2020_WS2812_LED
- removed IC1, IC2, IC3, IC4, IC5: SN74HC165PWR, Component_lib:SOP65P640X120-16N, symbol Component_lib:SN74HC165PWR
- removed IC7: ESP32-S2FH4, Component_lib:QFN40P700X700X90-57N-D, symbol Component lib:ESP32-S2FH4
- removed J10: USB_C_Receptacle_USB2.0, symbol Connector:USB_C_Receptacle_USB2.0
- removed L1: L, Inductor_SMD:L_0201_0603Metric, symbol Component lib:L
- removed R1: 0k, Resistor_SMD:R_0201_0603Metric, symbol Component lib:R
- removed R10, R11: 5.1k, Resistor_SMD:R_0201_0603Metric, symbol Component lib:R
- removed R2: 0, Resistor_SMD:R_0201_0603Metric, symbol Component lib:R
- removed R3, R5: 10k, Resistor_SMD:R_0201_0603Metric, symbol Component lib:R
- removed R4: 2k, Resistor_SMD:R_0201_0603Metric, symbol Component lib:R
- removed RN1, RN2, RN3, RN4, RN5: EXB-2HV103JV, Component_lib:EXB2HV_1, symbol Component lib:EXB-2HV103JV
- removed S1, S2: SKRPABE010, Component_lib:SKRPABE010, symbol Component lib:SKRPABE010
- removed SW1, SW10, SW11, SW12, SW13, SW14, SW15, SW16, SW17, SW18, SW19, SW2, SW20, SW21, SW22, SW23, SW24, SW25, SW26, SW27, SW28, SW29, SW3, SW30, SW31, SW32, SW33, SW34, SW35, SW36, SW37, SW38, SW39, SW4, SW40, SW5, SW6, SW7, SW8, SW9: SW_Push, Component_lib:Kailh_socket_PG1350_reversible, symbol Switch:SW_Push
- removed U1, U2: MIC5528-3.3YMT-T5, Component_lib:SON40P120X120X60-7N-D, symbol Component lib:MIC5528-3.3YMT-T5
- removed Y1: 40MHz, Component_lib:Crystal_SMD_2016-4Pin_2.0x1.6mm, symbol Device:Crystal_GND23_Small
Connections:
- no-connect marks 15 -> 0
Other:
- added sheet 100- Connectors (Connectors.kicad_sch)
- added sheet 200- Power (Power.kicad_sch)
- added sheet 300- 1S_Charger (1S_Charger.kicad_sch)
- added sheet 400- ESP32S2FH4S2 (ESP32S2FH4S2.kicad_sch)
- added sheet 500- Shift Register - Switch (ShiftRegisterSwitch.kicad_sch)
- added sheet 600- LEDs (LEDs.kicad_sch)
- note removed: "10-USB"
- note removed: "20-Power"
- note removed: "30-ESP32"
- note removed: "40MHz 10ppm"
- note removed: "Boot mode"
- note removed: "Reset"

Commit message: Worked on hierachic page again
Other:
- sheet 200- Power renamed 300- Power
- sheet 300- 1S_Charger renamed 200- 1S_Charger
- sheet 100- Connectors ports: added D+, D-, GND, VBUS; removed none
- sheet 200- 1S_Charger ports: added GND, VBAT, VBUS, VSYS; removed none
- sheet 300- Power ports: added +3V3, GND, LED_EN, VDD, VSYS; removed none

Commit message: Worked on hierachic sheet
Other:
- sheet 100- Connectors ports: added VBAT; removed none
- sheet 400- ESP32S2FH4S2 ports: added +3V3, D+, D-, GND, LED_MOSI, SR_CLK, SR_CS, SR_MISO; removed none

Commit message: Again on hierachic sheet
Other:
- sheet 400- ESP32S2FH4S2 ports: added LED_EN, PL; removed none
- sheet 500- Shift Register - Switch ports: added +3V3, CE, GND, PL, SPI_CLK, SPI_MISO; removed none
- sheet 600- LEDs ports: added GND, LED_MOSI, VDD; removed none
