File: Hardware/PMK_Keyboard/ShiftRegisterSwitch.kicad_sch (KiCad schematic)
At the start: 50 parts

Commit message: Worked on hierachic page again
Parts:
- U501, U502, U503, U504, U505: renamed from IC?; footprint Component_lib:SOP65P640X120-16N -> SOP65P640X120-16N
- gave numbers to parts that had none: 45
Connections:
- net 1: now also SW501.1; no longer SW509.1
- net 10: now also SW510.1; no longer SW518.1
- net 11: now also SW511.1; no longer SW519.1
- net 12: now also SW512.1; no longer SW520.1
- net 13: now also SW513.1; no longer SW521.1
- net 14: now also SW514.1; no longer SW522.1
- net 15: now also SW515.1; no longer SW523.1
- net 16: now also SW516.1; no longer SW524.1
- net 17: now also SW517.1; no longer SW525.1
- net 18: now also SW518.1; no longer SW526.1
- net 19: now also SW519.1; no longer SW527.1
- net 2: now also SW502.1; no longer SW510.1
- net 20: now also SW520.1; no longer SW528.1
- net 21: now also SW521.1; no longer SW529.1
- net 22: now also SW522.1; no longer SW530.1
- net 23: now also SW523.1; no longer SW531.1
- net 24: now also SW524.1; no longer SW532.1
- net 25: now also SW525.1; no longer SW501.1
- net 26: now also SW526.1; no longer SW502.1
- net 27: now also SW527.1; no longer SW503.1
- net 28: now also SW528.1; no longer SW504.1
- net 29: now also SW529.1; no longer SW505.1
- net 3: now also SW503.1; no longer SW511.1
- net 30: now also SW530.1; no longer SW506.1
- net 31: now also SW531.1; no longer SW507.1
- net 32: now also SW532.1; no longer SW508.1
- net 4: now also SW504.1; no longer SW512.1
- net 5: now also SW505.1; no longer SW513.1
- net 6: now also SW506.1; no longer SW514.1
- net 7: now also SW507.1; no longer SW515.1
- net 8: now also SW508.1; no longer SW516.1
- net 9: now also SW509.1; no longer SW517.1
Other:
- moved on the sheet: SW501, SW502, SW503, SW504, SW505, SW506, SW507, SW508, SW509, SW510, SW511, SW512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

Commit message: Again on hierachic sheet
Other:
- company: (none) -> PumaCorp
- title: (none) -> PMK_Keyboard
- moved on the sheet: RN501, RN502, RN503, RN504, RN505, SW501, SW502, SW503, SW504, SW505, SW506, SW507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

Commit message: Schematic is done, only possible update is change of ESP pins
Other:
- moved on the sheet: RN501, RN502, RN503, RN504, RN505, SW501, SW502, SW503, SW504, SW505, SW506, SW507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

Commit message: Routing is finally updated
Parts:
- U501, U502, U503, U504, U505: footprint SOP65P640X120-16N -> Component_lib:SOP65P640X120-16N
Changed lines of the file:
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@@
       (effects (font (size 1.27 1.27)) (justify right))
     )
-    (property "Footprint" "SOP65P640X120-16N" (id 2) (at 307.34 132.08 0)
+    (property "Footprint" "Component_lib:SOP65P640X120-16N" (id 2) (at 307.34 132.08 0)
       (effects (font (size 1.27 1.27)) (justify left) hide)
     )
@@
       (effects (font (size 1.27 1.27)) (justify right))
     )
-    (property "Footprint" "SOP65P640X120-16N" (id 2) (at 53.34 132.08 0)
+    (property "Footprint" "Component_lib:SOP65P640X120-16N" (id 2) (at 53.34 132.08 0)
       (effects (font (size 1.27 1.27)) (justify left) hide)
     )
@@
       (effects (font (size 1.27 1.27)) (justify right))
     )
-    (property "Footprint" "SOP65P640X120-16N" (id 2) (at 243.84 132.08 0)
+    (property "Footprint" "Component_lib:SOP65P640X120-16N" (id 2) (at 243.84 132.08 0)
       (effects (font (size 1.27 1.27)) (justify left) hide)
     )
@@
       (effects (font (size 1.27 1.27)) (justify right))
     )
-    (property "Footprint" "SOP65P640X120-16N" (id 2) (at 116.84 132.08 0)
+    (property "Footprint" "Component_lib:SOP65P640X120-16N" (id 2) (at 116.84 132.08 0)
       (effects (font (size 1.27 1.27)) (justify left) hide)
     )
@@
       (effects (font (size 1.27 1.27)) (justify right))
     )
-    (property "Footprint" "SOP65P640X120-16N" (id 2) (at 180.34 132.08 0)
-      (effects (font (size 1.27 1.27)) (justify left) hide)
-    )
+    (property "Footprint" "Component_lib:SOP65P640X120-16N" (id 2) (at 180.34 132.08 0)
+      (effects (font (size 1.27 1.27)) (justify left) hide)
+    )

Commit message: Routing is almost done
Parts:
- SW501: footprint Component_lib:Kailh_socket_PG1350_reversible -> Component_lib:SKRPABE010
