File: Hardware/PMK_Dongle/PMK_Dongle/PMK_Dongle.kicad_sch (KiCad schematic)
At the start: 31 parts, among them IC1 ESP32-S2FH4, J1 USB_A, U1 MIC5528-3.3YMT-T5, Y1 40MHz

Commit message: Routing is almost done, just need to check quartz
Connections:
- net QUARTZ_1: now also IC1.53 (XTAL_P), Y1.4; no longer R1.1, Y1.1
- net QUARTZ_2: now also R1.1, Y1.1; no longer IC1.52 (XTAL_N), Y1.4
- net QUARTZ_3: now also IC1.52 (XTAL_N); no longer IC1.53 (XTAL_P)
Other:
- moved on the sheet: C4, R1
Changed lines of the file:
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@@
+    (stroke (width 0) (type default) (color 0 0 0 0))
+  )
+  (wire (pts (xy 116.84 157.48) (xy 124.46 157.48))
     (stroke (width 0) (type default) (color 0 0 0 0))
   )
@@
     (stroke (width 0) (type default) (color 0 0 0 0))
   )
-  (wire (pts (xy 116.84 157.48) (xy 116.84 175.26))
-    (stroke (width 0) (type default) (color 0 0 0 0))
-  )
   (wire (pts (xy 53.34 205.74) (xy 63.5 205.74))
     (stroke (width 0) (type default) (color 0 0 0 0))
@@
     (stroke (width 0) (type default) (color 0 0 0 0))
   )
+  (wire (pts (xy 124.46 157.48) (xy 124.46 160.02))
+    (stroke (width 0) (type default) (color 0 0 0 0))
+  )
   (wire (pts (xy 134.62 66.04) (xy 134.62 68.58))
     (stroke (width 0) (type default) (color 0 0 0 0))
   )
+  (wire (pts (xy 116.84 172.72) (xy 116.84 175.26))
+    (stroke (width 0) (type default) (color 0 0 0 0))
+  )
   (wire (pts (xy 254 231.14) (xy 254 233.68))
     (stroke (width 0) (type default) (color 0 0 0 0))
@@
     (stroke (width 0) (type default) (color 0 0 0 0))
   )
-  (wire (pts (xy 121.92 157.48) (xy 116.84 157.48))
+  (wire (pts (xy 114.3 157.48) (xy 116.84 157.48))
     (stroke (width 0) (type default) (color 0 0 0 0))
   )
@@
     (stroke (width 0) (type default) (color 0 0 0 0))
   )
-  (wire (pts (xy 114.3 157.48) (xy 116.84 157.48))
-    (stroke (width 0) (type default) (color 0 0 0 0))
-  )
   (wire (pts (xy 53.34 180.34) (xy 53.34 177.8))
     (stroke (width 0) (type default) (color 0 0 0 0))
@@
     (stroke (width 0) (type default) (color 0 0 0 0))
   )
-  (wire (pts (xy 104.14 175.26) (xy 104.14 172.72))
-    (stroke (width 0) (type default) (color 0 0 0 0))
-  )
   (wire (pts (xy 73.66 182.88) (xy 73.66 185.42))
     (stroke (width 0) (type default) (color 0 0 0 0))
@@
     (stroke (width 0) (type default) (color 0 0 0 0))
   )
-  (wire (pts (xy 104.14 165.1) (xy 104.14 157.48))
-    (stroke (width 0) (type default) (color 0 0 0 0))
-  )
-  (wire (pts (xy 121.92 167.64) (xy 121.92 170.18))
+  (wire (pts (xy 104.14 157.48) (xy 104.14 175.26))
+    (stroke (width 0) (type default) (color 0 0 0 0))
+  )
+  (wire (pts (xy 124.46 167.64) (xy 124.46 170.18))
     (stroke (width 0) (type default) (color 0 0 0 0))
   )
@@
     (stroke (width 0) (type default) (color 0 0 0 0))
   )
+  (wire (pts (xy 116.84 157.48) (xy 116.84 165.1))
+    (stroke (width 0) (type default) (color 0 0 0 0))
+  )
   (wire (pts (xy 86.36 208.28) (xy 86.36 205.74))
     (stroke (width 0) (type default) (color 0 0 0 0))
@@
   )
   (wire (pts (xy 165.1 175.26) (xy 165.1 177.8))
-    (stroke (width 0) (type default) (color 0 0 0 0))
-  )
-  (wire (pts (xy 121.92 160.02) (xy 121.92 157.48))
     (stroke (width 0) (type default) (color 0 0 0 0))
   )
@@
     (effects (font (size 1.27 1.27)) (justify left bottom))
   )
-  (label "QUARTZ_3" (at 104.14 175.26 0)
+  (label "QUARTZ_3" (at 111.76 175.26 0)
     (effects (font (size 1.27 1.27)) (justify left bottom))
   )
@@
   )
   (symbol (lib_id "power:GND") (at 111.76 152.4 180) (unit 1)
-    (in_bom yes) (on_board yes) (fields_autoplaced)
+    (in_bom yes) (on_board yes)
     (property "Reference" "#PWR0120" (id 0) (at 111.76 146.05 0)
       (effects (font (size 1.27 1.27)) hide)
     )
-    (property "Value" "GND" (id 1) (at 113.665 151.5638 0)
+    (property "Value" "GND" (id 1) (at 106.68 152.4 0)
       (effects (font (size 1.27 1.27)) (justify right))
     )
@@
     (pin "2")
   )
-  (symbol (lib_id "Component lib:C") (at 121.92 160.02 0) (unit 1)
-    (in_bom yes) (on_board yes) (fields_autoplaced)
-    (property "Reference" "C4" (id 0) (at 124.841 162.9953 0)
-      (effects (font (size 1.27 1.27)) (justify left))
-    )
-    (property "Value" "15p" (id 1) (at 124.841 165.5322 0)
-      (effects (font (size 1.27 1.27)) (justify left))
-    )
-    (property "Footprint" "Capacitor_SMD:C_0201_0603Metric" (id 2) (at 122.8852 167.64 0)
-      (effects (font (size 1.27 1.27)) hide)
-    )
-    (property "Datasheet" "~" (id 3) (at 121.92 163.83 0)
+  (symbol (lib_id "Component lib:C") (at 124.46 160.02 0) (unit 1)
+    (in_bom yes) (on_board yes) (fields_autoplaced)
+    (property "Reference" "C4" (id 0) (at 127.381 162.9953 0)
+      (effects (font (size 1.27 1.27)) (justify left))
+    )
+    (property "Value" "15p" (id 1) (at 127.381 165.5322 0)
+      (effects (font (size 1.27 1.27)) (justify left))
+    )
+    (property "Footprint" "Capacitor_SMD:C_0201_0603Metric" (id 2) (at 125.4252 167.64 0)
+      (effects (font (size 1.27 1.27)) hide)
+    )
+    (property "Datasheet" "~" (id 3) (at 124.46 163.83 0)
       (effects (font (size 1.27 1.27)) hide)
     )
@@
     (pin "1")
   )
-  (symbol (lib_id "Component lib:R") (at 104.14 165.1 0) (unit 1)
-    (in_bom yes) (on_board yes) (fields_autoplaced)
-    (property "Reference" "R1" (id 0) (at 105.918 168.0753 0)
-      (effects (font (size 1.27 1.27)) (justify left))
-    )
-    (property "Value" "0" (id 1) (at 105.918 170.6122 0)
-      (effects (font (size 1.27 1.27)) (justify left))
-    )
-    (property "Footprint" "Resistor_SMD:R_0201_0603Metric" (id 2) (at 102.362 168.91 90)
-      (effects (font (size 1.27 1.27)) hide)
-    )
-    (property "Datasheet" "~" (id 3) (at 104.14 168.91 0)
+  (symbol (lib_id "Component lib:R") (at 116.84 165.1 0) (unit 1)
+    (in_bom yes) (on_board yes) (fields_autoplaced)
+    (property "Reference" "R1" (id 0) (at 118.618 168.0753 0)
+      (effects (font (size 1.27 1.27)) (justify left))
+    )
+    (property "Value" "0" (id 1) (at 118.618 170.6122 0)
+      (effects (font (size 1.27 1.27)) (justify left))
+    )
+    (property "Footprint" "Resistor_SMD:R_0201_0603Metric" (id 2) (at 115.062 168.91 90)
+      (effects (font (size 1.27 1.27)) hide)
+    )
+    (property "Datasheet" "~" (id 3) (at 116.84 168.91 0)
       (effects (font (size 1.27 1.27)) hide)
     )
@@
     (pin "1")
   )
-  (symbol (lib_id "Device:Crystal_GND23_Small") (at 111.76 157.48 0) (unit 1)
+  (symbol (lib_id "Device:Crystal_GND23_Small") (at 111.76 157.48 0) (mirror y) (unit 1)
     (in_bom yes) (on_board yes)
-    (property "Reference" "Y1" (id 0) (at 101.6 149.86 0))
-    (property "Value" "40MHz" (id 1) (at 104.14 152.4 0))
+    (property "Reference" "Y1" (id 0) (at 121.92 149.86 0))
+    (property "Value" "40MHz" (id 1) (at 119.38 152.4 0))
     (property "Footprint" "Component_lib:NX2016SA32MEXS00ACS06465" (id 2) (at 111.76 157.48 0)
       (effects (font (size 1.27 1.27)) hide)
@@
     (pin "2")
   )
-  (symbol (lib_id "power:GND") (at 121.92 170.18 0) (unit 1)
-    (in_bom yes) (on_board yes) (fields_autoplaced)
-    (property "Reference" "#PWR0128" (id 0) (at 121.92 176.53 0)
-      (effects (font (size 1.27 1.27)) hide)
-    )
-    (property "Value" "GND" (id 1) (at 121.92 174.6234 0))
-    (property "Footprint" "" (id 2) (at 121.92 170.18 0)
-      (effects (font (size 1.27 1.27)) hide)
-    )
-    (property "Datasheet" "" (id 3) (at 121.92 170.18 0)
-      (effects (font (size 1.27 1.27)) hide)
-    )
+  (symbol (lib_id "power:GND") (at 124.46 170.18 0) (unit 1)
+    (in_bom yes) (on_board yes) (fields_autoplaced)
+    (property "Reference" "#PWR0128" (id 0) (at 124.46 176.53 0)
+      (effects (font (size 1.27 1.27)) hide)
+    )
+    (property "Value" "GND" (id 1) (at 124.46 174.6234 0))
+    (property "Footprint" "" (id 2) (at 124.46 170.18 0)
+      (effects (font (size 1.27 1.27)) hide)
+    )
+    (property "Datasheet" "" (id 3) (at 124.46 170.18 0)
+      (effects (font (size 1.27 1.27)) hide)
+    )

Commit message: Routing is done
Parts:
- removed Y1: 40MHz, Component_lib:NX2016SA32MEXS00ACS06465, symbol Device:Crystal_GND23_Small
- added Y1: Crystal_GND24_Small, Component_lib:Crystal_SMD_2016-4Pin_2.0x1.6mm, symbol Device:Crystal_GND24_Small
Connections:
- net GND: now also Y1.2, Y1.4
- net QUARTZ_1: now also R1.1, Y1.1; no longer IC1.53 (XTAL_P)
- net QUARTZ_2: now also IC1.52 (XTAL_N), Y1.3; no longer R1.1
- net QUARTZ_3: now also IC1.53 (XTAL_P); no longer IC1.52 (XTAL_N)
Other:
- moved on the sheet: R1
