File: Hardware/PMK_Keyboard/PMK_Keyboard_HW01/Connectors.kicad_sch (KiCad schematic)
At the start: 4 parts, among them J101 USB4510-03-1-A

Commit message: Working on schematic
Parts:
- added J113: Cirque, Component_lib:Cirque trackpad, symbol Connector:Conn_01x14_Female
- added J602: Conn_01x05_Pin, symbol Connector:Conn_01x05_Pin
Connections:
- net GND: now also J113.11 (Pin_11), J602.5 (Pin_5)
- new net 3V3: J113.12 (Pin_12), J602.1 (Pin_1)
- new net INT: J602.4 (Pin_4)
- new net MISO: J113.2 (Pin_2)
- new net MOSI: J113.5 (Pin_5)
- new net NCS: J113.3 (Pin_3)
- new net SCL: J113.9 (Pin_9), J602.3 (Pin_3)
- new net SCLK: J113.1 (Pin_1)
- new net SDA: J113.10 (Pin_10), J602.2 (Pin_2)
- no-connect marks 2 -> 8
Other:
- note added: "200- Connectors"
- note added: "For 3D mouse LDC1612"
- note added: "For trackpad Cirque FPC"
- note removed: "100-USB"
Changed lines of the file:
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@@
   (junction (at 66.04 63.5) (diameter 0) (color 0 0 0 0)
   )
+  (no_connect (at 231.14 86.36))
   (no_connect (at 63.5 81.28))
   (no_connect (at 63.5 78.74))
+  (no_connect (at 231.14 106.68))
+  (no_connect (at 231.14 83.82))
+  (no_connect (at 231.14 88.9))
+  (no_connect (at 231.14 93.98))
+  (no_connect (at 231.14 104.14))
   (wire (pts (xy 271.78 20.32) (xy 271.78 22.86))
     (stroke (width 0) (type default))
   )
+  (wire (pts (xy 228.6 73.66) (xy 231.14 73.66))
+    (stroke (width 0) (type default))
+  )
   (wire (pts (xy 63.5 58.42) (xy 83.82 58.42))
     (stroke (width 0) (type default))
@@
     (stroke (width 0) (type default))
   )
+  (wire (pts (xy 228.6 76.2) (xy 231.14 76.2))
+    (stroke (width 0) (type default))
+  )
+  (wire (pts (xy 226.06 81.28) (xy 231.14 81.28))
+    (stroke (width 0) (type default))
+  )
   (wire (pts (xy 271.78 27.94) (xy 271.78 30.48))
     (stroke (width 0) (type default))
@@
     (stroke (width 0) (type default))
   )
+  (wire (pts (xy 226.06 96.52) (xy 231.14 96.52))
+    (stroke (width 0) (type default))
+  )
   (wire (pts (xy 271.78 22.86) (xy 274.32 22.86))
     (stroke (width 0) (type default))
   )
+  (wire (pts (xy 162.56 73.66) (xy 165.1 73.66))
+    (stroke (width 0) (type default))
+  )
   (wire (pts (xy 93.98 55.88) (xy 93.98 60.96))
     (stroke (width 0) (type default))
@@
     (stroke (width 0) (type default))
   )
+  (wire (pts (xy 162.56 71.12) (xy 165.1 71.12))
+    (stroke (width 0) (type default))
+  )
   (wire (pts (xy 63.5 68.58) (xy 66.04 68.58))
     (stroke (width 0) (type default))
   )
+  (wire (pts (xy 162.56 78.74) (xy 165.1 78.74))
+    (stroke (width 0) (type default))
+  )
   (wire (pts (xy 63.5 55.88) (xy 93.98 55.88))
     (stroke (width 0) (type default))
@@
     (stroke (width 0) (type default))
   )
+  (wire (pts (xy 162.56 76.2) (xy 165.1 76.2))
+    (stroke (width 0) (type default))
+  )
   (wire (pts (xy 271.78 45.72) (xy 274.32 45.72))
     (stroke (width 0) (type default))
@@
     (stroke (width 0) (type default))
   )
+  (wire (pts (xy 162.56 83.82) (xy 162.56 81.28))
+    (stroke (width 0) (type default))
+  )
+  (wire (pts (xy 162.56 81.28) (xy 165.1 81.28))
+    (stroke (width 0) (type default))
+  )
   (wire (pts (xy 63.5 66.04) (xy 66.04 66.04))
     (stroke (width 0) (type default))
   )
+  (wire (pts (xy 226.06 101.6) (xy 231.14 101.6))
+    (stroke (width 0) (type default))
+  )
   (wire (pts (xy 48.26 129.54) (xy 48.26 132.08))
     (stroke (width 0) (type default))
@@
     (stroke (width 0) (type default))
   )
+  (wire (pts (xy 226.06 91.44) (xy 231.14 91.44))
+    (stroke (width 0) (type default))
+  )
+  (wire (pts (xy 228.6 76.2) (xy 228.6 109.22))
+    (stroke (width 0) (type default))
+  )
+  (wire (pts (xy 226.06 78.74) (xy 231.14 78.74))
+    (stroke (width 0) (type default))
+  )
   (wire (pts (xy 50.8 86.36) (xy 50.8 88.9))
     (stroke (width 0) (type default))
   )
+  (wire (pts (xy 226.06 99.06) (xy 231.14 99.06))
+    (stroke (width 0) (type default))
+  )
   (wire (pts (xy 271.78 35.56) (xy 274.32 35.56))
     (stroke (width 0) (type default))
@@
     (stroke (width 0) (type default))
   )
-  (text "100-USB" (at 15.24 30.48 0)
+  (text "200- Connectors" (at 15.24 30.48 0)
     (effects (font (size 8 8) (thickness 3) bold) (justify left bottom))
+  )
+  (text "For trackpad\nCirque FPC" (at 226.06 68.58 0)
+    (effects (font (size 1.27 1.27)) (justify left bottom))
+  )
+  (text "For 3D mouse\nLDC1612" (at 160.02 66.04 0)
+    (effects (font (size 1.27 1.27)) (justify left bottom))
+  )
+  (label "INT" (at 162.56 78.74 180) (fields_autoplaced)
+    (effects (font (size 1.27 1.27)) (justify right bottom))
   )
   (label "VBAT" (at 271.78 22.86 180) (fields_autoplaced)
@@
     (effects (font (size 1.27 1.27)) (justify left bottom))
   )
+  (label "3V3" (at 162.56 71.12 180) (fields_autoplaced)
+    (effects (font (size 1.27 1.27)) (justify right bottom))
+  )
+  (label "3V3" (at 228.6 73.66 180) (fields_autoplaced)
+    (effects (font (size 1.27 1.27)) (justify right bottom))
+  )
+  (label "SCL" (at 162.56 76.2 180) (fields_autoplaced)
+    (effects (font (size 1.27 1.27)) (justify right bottom))
+  )
+  (label "SCL" (at 226.06 81.28 180) (fields_autoplaced)
+    (effects (font (size 1.27 1.27)) (justify right bottom))
+  )
   (label "CC2" (at 73.66 58.42 0) (fields_autoplaced)
     (effects (font (size 1.27 1.27)) (justify left bottom))
@@
     (effects (font (size 1.27 1.27)) (justify right bottom))
   )
+  (label "MOSI" (at 226.06 91.44 180) (fields_autoplaced)
+    (effects (font (size 1.27 1.27)) (justify right bottom))
+  )
+  (label "SDA" (at 226.06 78.74 180) (fields_autoplaced)
+    (effects (font (size 1.27 1.27)) (justify right bottom))
+  )
+  (label "SDA" (at 162.56 73.66 180) (fields_autoplaced)
+    (effects (font (size 1.27 1.27)) (justify right bottom))
+  )
+  (label "NCS" (at 226.06 96.52 180) (fields_autoplaced)
+    (effects (font (size 1.27 1.27)) (justify right bottom))
+  )
+  (label "SCLK" (at 226.06 101.6 180) (fields_autoplaced)
+    (effects (font (size 1.27 1.27)) (justify right bottom))
+  )
   (label "D-" (at 271.78 35.56 180) (fields_autoplaced)
     (effects (font (size 1.27 1.27)) (justify right bottom))
@@
   (label "CC1" (at 73.66 55.88 0) (fields_autoplaced)
     (effects (font (size 1.27 1.27)) (justify left bottom))
+  )
+  (label "MISO" (at 226.06 99.06 180) (fields_autoplaced)
+    (effects (font (size 1.27 1.27)) (justify right bottom))
   )
   (label "VBAT" (at 48.26 132.08 0) (fields_autoplaced)
@@
     )
   )
+  (symbol (lib_id "power:GND") (at 162.56 83.82 0) (unit 1)
+    (in_bom yes) (on_board yes) (dnp no) (fields_autoplaced)
+    (property "Reference" "#PWR0683" (at 162.56 90.17 0)
+      (effects (font (size 1.27 1.27)) hide)
+    )
+    (property "Value" "GND" (at 162.56 88.2634 0)
+      (effects (font (size 1.27 1.27)))
+    )
+    (property "Footprint" "" (at 162.56 83.82 0)
+      (effects (font (size 1.27 1.27)) hide)
+    )
+    (property "Datasheet" "" (at 162.56 83.82 0)
+      (effects (font (size 1.27 1.27)) hide)
+    )
+    (pin "1")
+    (instances
+      (project "PMK_Keyboard_HW01"
+        (path "/c3b08055-08a5-4979-9bf8-f36ab0917722/cf9fd53d-a626-44ae-9c40-26b02d8cda14"
+          (reference "#PWR0683") (unit 1)
+        )
+        (path "/c3b08055-08a5-4979-9bf8-f36ab0917722/f4bd3789-d94c-4771-8f5c-2a22000e96d6"
+          (reference "#PWR0688") (unit 1)
+        )
+      )
+    )
+  )
   (symbol (lib_id "power:GND") (at 50.8 88.9 0) (unit 1)
     (in_bom yes) (on_board yes) (dnp no) (fields_autoplaced)
@@
     )
   )
+  (symbol (lib_id "Connector:Conn_01x14_Female") (at 236.22 88.9 0) (unit 1)
+    (in_bom yes) (on_board yes) (dnp no) (fields_autoplaced)
+    (property "Reference" "J113" (at 238.125 88.8999 0)
+      (effects (font (size 1.27 1.27)) (justify left))
+    )
+    (property "Value" "Cirque" (at 238.125 91.4399 0)
+      (effects (font (size 1.27 1.27)) (justify left))
+    )
+    (property "Footprint" "Component_lib:Cirque trackpad" (at 257.81 85.09 0)
+      (effects (font (size 1.27 1.27)) hide)
+    )
+    (property "Datasheet" "~" (at 236.22 88.9 0)
+      (effects (font (size 1.27 1.27)) hide)
+    )
+    (pin "1")
+    (pin "10")
+    (pin "11")
+    (pin "12")
+    (pin "13")
+    (pin "14")
+    (pin "2")
+    (pin "3")
+    (pin "4")
+    (pin "5")
+    (pin "6")
+    (pin "7")
+    (pin "8")
+    (pin "9")
+    (instances
+      (project "dilemma"
+        (path "/7353e96a-343a-4876-b497-b1d205a14d97"
+          (reference "J113") (unit 1)
+        )
+      )
+      (project "PMK_Keyboard_HW01"
+        (path "/c3b08055-08a5-4979-9bf8-f36ab0917722/cf9fd53d-a626-44ae-9c40-26b02d8cda14"
+          (reference "J601") (unit 1)
+        )
+      )
+    )
+  )
   (symbol (lib_id "power:GND") (at 93.98 71.12 0) (unit 1)
     (in_bom yes) (on_board yes) (dnp no) (fields_autoplaced)
@@
         (path "/c3b08055-08a5-4979-9bf8-f36ab0917722/f4bd3789-d94c-4771-8f5c-2a22000e96d6"
           (reference "R602") (unit 1)
+        )
+      )
+    )
+  )
+  (symbol (lib_id "power:GND") (at 228.6 109.22 0) (unit 1)
+    (in_bom yes) (on_board yes) (dnp no) (fields_autoplaced)
+    (property "Reference" "#PWR0688" (at 228.6 115.57 0)
+      (effects (font (size 1.27 1.27)) hide)
+    )
+    (property "Value" "GND" (at 228.6 113.6634 0)
+      (effects (font (size 1.27 1.27)))
+    )
+    (property "Footprint" "" (at 228.6 109.22 0)
+      (effects (font (size 1.27 1.27)) hide)
+    )
+    (property "Datasheet" "" (at 228.6 109.22 0)
+      (effects (font (size 1.27 1.27)) hide)
+    )
+    (pin "1")
+    (instances
+      (project "PMK_Keyboard_HW01"
+        (path "/c3b08055-08a5-4979-9bf8-f36ab0917722/cf9fd53d-a626-44ae-9c40-26b02d8cda14"
+          (reference "#PWR0688") (unit 1)
+        )
+        (path "/c3b08055-08a5-4979-9bf8-f36ab0917722/f4bd3789-d94c-4771-8f5c-2a22000e96d6"
+          (reference "#PWR0688") (unit 1)
         )
       )
@@
         )
       )
+    )
+  )
+  (symbol (lib_id "Connector:Conn_01x05_Pin") (at 170.18 76.2 0) (mirror y) (unit 1)
+    (in_bom yes) (on_board yes) (dnp no) (fields_autoplaced)
+    (property "Reference" "J602" (at 170.8912 75.5563 0)
+      (effects (font (size 1.27 1.27)) (justify right))
+    )
+    (property "Value" "Conn_01x05_Pin" (at 170.8912 77.4773 0)
+      (effects (font (size 1.27 1.27)) (justify right))
+    )
+    (property "Footprint" "" (at 170.18 76.2 0)
+      (effects (font (size 1.27 1.27)) hide)
+    )
+    (property "Datasheet" "~" (at 170.18 76.2 0)
+      (effects (font (size 1.27 1.27)) hide)
+    )
+    (pin "1")
+    (pin "2")
+    (pin "3")
+    (pin "4")
+    (pin "5")
+    (instances
+      (project "PMK_Keyboard_HW01"
+        (path "/c3b08055-08a5-4979-9bf8-f36ab0917722/cf9fd53d-a626-44ae-9c40-26b02d8cda14"
+          (reference "J602") (unit 1)
+        )
+      )

Commit message: Started routing
Parts:
- removed BT101: Battery_Cell, Component_lib:BatteryHolder_Keystone_1042_1x18650_DUALSIDE, symbol Device:Battery_Cell
- added J204: S2B-PH-SM4-TB, Component_lib:JST_PH_B2B-PH-SM4-TB_1x02-1MP_P2.00mm_Vertical_DUALSIDE, symbol Component_lib:S2B-PH-SM4-TB
- added R203, R204: 0, Resistor_SMD:R_0201_0603Metric, symbol Component lib:R
- added SW201: 450405020524, Component_lib:450405020524_DUALSIDE, symbol Component_lib:450405020524
- J202: renamed from J602; footprint (none) -> Component_lib:SMD_CONN_01x5_1.5mm
- renumbered J101 to J201, R101 to R201, R102 to R202
Connections:
- net GND: now also J204.2 (Pin_2), J204.MP (MountPin)
- net VBAT: now also R203.2, R204.2
- new net: R203.1, SW201.1 (A)
- new net: R204.1, SW201.2 (C)
- new net: J204.1 (Pin_1), SW201.3 (B)
Other:
- moved on the sheet: J113

Commit message: working on routing
Parts:
- J204: footprint Component_lib:JST_PH_B2B-PH-SM4-TB_1x02-1MP_P2.00mm_Vertical_DUALSIDE -> Component_lib:JST_PH_S2B-PH-SM4-TB_1x02-1MP_P2.00mm_Horizontal_DUALSIDE
Changed lines of the file:
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@@
       (effects (font (size 1.27 1.27)))
     )
-    (property "Footprint" "Component_lib:JST_PH_B2B-PH-SM4-TB_1x02-1MP_P2.00mm_Vertical_DUALSIDE" (at 58.42 139.7 0)
+    (property "Footprint" "Component_lib:JST_PH_S2B-PH-SM4-TB_1x02-1MP_P2.00mm_Horizontal_DUALSIDE" (at 58.42 139.7 0)
       (effects (font (size 1.27 1.27)) hide)
     )

Commit message: a bit of routing
Parts:
- removed J113: Cirque, Component_lib:Cirque trackpad, symbol Connector:Conn_01x14_Female
- added J301: 505110-1292, 5051101292, symbol Component_lib:505110-1292
Connections:
- net 3V3: now also J301.12
- net GND: now also J301.11, J301.MP1, J301.MP2
- net MISO: now also J301.2
- net MOSI: now also J301.5
- net NCS: now also J301.3
- net SCL: now also J301.9
- net SCLK: now also J301.1
- net SDA: now also J301.10
- new net BTN1: J301.8
- new net BTN2: J301.7
- new net BTN3: J301.6
- new net DR: J301.4
- no-connect marks 8 -> 2

Commit message: Need to add some silkscreenthen done!
Parts:
- J301: footprint 5051101292 -> Component_lib:5051101292
- R201, R202, R203, R204: footprint Resistor_SMD:R_0201_0603Metric -> Resistor_SMD:R_0402_1005Metric
Connections:
- net BTN1 renamed GP_CE
Changed lines of the file:
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@@
+    (stroke (width 0) (type default))
+  )
+  (wire (pts (xy 271.78 86.36) (xy 274.32 86.36))
     (stroke (width 0) (type default))
   )
@@
     (stroke (width 0) (type default))
   )
-  (wire (pts (xy 271.78 88.9) (xy 271.78 86.36))
+  (wire (pts (xy 271.78 93.98) (xy 271.78 91.44))
     (stroke (width 0) (type default))
   )
@@
     (stroke (width 0) (type default))
   )
-  (wire (pts (xy 271.78 86.36) (xy 274.32 86.36))
+  (wire (pts (xy 271.78 91.44) (xy 274.32 91.44))
     (stroke (width 0) (type default))
   )
@@
     (effects (font (size 1.27 1.27)) (justify left bottom))
   )
-  (label "BTN1" (at 200.66 81.28 180) (fields_autoplaced)
+  (label "GP_CE" (at 200.66 81.28 180) (fields_autoplaced)
     (effects (font (size 1.27 1.27)) (justify right bottom))
   )
@@
     (effects (font (size 1.27 1.27)) (justify left bottom))
   )
+  (label "GP_CE" (at 271.78 86.36 180) (fields_autoplaced)
+    (effects (font (size 1.27 1.27)) (justify right bottom))
+  )
   (label "VBUS" (at 271.78 30.48 180) (fields_autoplaced)
     (effects (font (size 1.27 1.27)) (justify right bottom))
@@
     (effects (font (size 1.27 1.27)) (justify left))
   )
-  (hierarchical_label "GND" (shape passive) (at 274.32 86.36 0) (fields_autoplaced)
+  (hierarchical_label "GP_CE" (shape input) (at 274.32 86.36 0) (fields_autoplaced)
+    (effects (font (size 1.27 1.27)) (justify left))
+  )
+  (hierarchical_label "GND" (shape passive) (at 274.32 91.44 0) (fields_autoplaced)
     (effects (font (size 1.27 1.27)) (justify left))
   )
@@
       (effects (font (size 1.27 1.27)) (justify left))
     )
-    (property "Footprint" "Resistor_SMD:R_0201_0603Metric" (at 82.042 64.77 90)
+    (property "Footprint" "Resistor_SMD:R_0402_1005Metric" (at 82.042 64.77 90)
       (effects (font (size 1.27 1.27)) hide)
     )
@@
       (effects (font (size 1.27 1.27)))
     )
-    (property "Footprint" "5051101292" (at 187.96 101.6 0)
+    (property "Footprint" "Component_lib:5051101292" (at 187.96 101.6 0)
       (effects (font (size 1.27 1.27)) (justify left) hide)
     )
@@
       (effects (font (size 1.27 1.27)))
     )
-    (property "Footprint" "Resistor_SMD:R_0201_0603Metric" (at 77.47 141.478 90)
+    (property "Footprint" "Resistor_SMD:R_0402_1005Metric" (at 77.47 141.478 90)
       (effects (font (size 1.27 1.27)) hide)
     )
@@
       (effects (font (size 1.27 1.27)))
     )
-    (property "Footprint" "Resistor_SMD:R_0201_0603Metric" (at 77.47 146.558 90)
+    (property "Footprint" "Resistor_SMD:R_0402_1005Metric" (at 77.47 146.558 90)
       (effects (font (size 1.27 1.27)) hide)
     )
@@
       (effects (font (size 1.27 1.27)) (justify left))
     )
-    (property "Footprint" "Resistor_SMD:R_0201_0603Metric" (at 92.202 64.77 90)
+    (property "Footprint" "Resistor_SMD:R_0402_1005Metric" (at 92.202 64.77 90)
       (effects (font (size 1.27 1.27)) hide)
     )
@@
     )
   )
-  (symbol (lib_id "power:GND") (at 271.78 88.9 0) (unit 1)
-    (in_bom yes) (on_board yes) (dnp no) (fields_autoplaced)
-    (property "Reference" "#PWR0208" (at 271.78 95.25 0)
-      (effects (font (size 1.27 1.27)) hide)
-    )
-    (property "Value" "GND" (at 271.78 93.3434 0)
-      (effects (font (size 1.27 1.27)))
-    )
-    (property "Footprint" "" (at 271.78 88.9 0)
-      (effects (font (size 1.27 1.27)) hide)
-    )
-    (property "Datasheet" "" (at 271.78 88.9 0)
-      (effects (font (size 1.27 1.27)) hide)
-    )
+  (symbol (lib_id "power:GND") (at 271.78 93.98 0) (unit 1)
+    (in_bom yes) (on_board yes) (dnp no) (fields_autoplaced)
+    (property "Reference" "#PWR0208" (at 271.78 100.33 0)
+      (effects (font (size 1.27 1.27)) hide)
+    )
+    (property "Value" "GND" (at 271.78 98.4234 0)
+      (effects (font (size 1.27 1.27)))
+    )
+    (property "Footprint" "" (at 271.78 93.98 0)
+      (effects (font (size 1.27 1.27)) hide)
+    )
+    (property "Datasheet" "" (at 271.78 93.98 0)
+      (effects (font (size 1.27 1.27)) hide)
+    )

Commit message: added mounting holes + fix in ref des
Parts:
- renumbered J201 to J303, J202 to J304, J301 to J305, J204 to J306, R201 to R303, R202 to R304, R203 to R305, R204 to R306, SW201 to SW301
Other:
- note added: "300- Connectors"
- note removed: "200- Connectors"
