File: Hardware/PMK_Keyboard/PMK_Keyboard_HW01/PMK_Keyboard_HW01.kicad_sch (KiCad schematic)
At the start: 0 parts

Commit message: started keyboard HW01
Other:
- removed sheet 200- 1S_Charger
- removed sheet 300- Power
- removed sheet 400- ESP32S2FH4S2
- added sheet 100- PSoM (PSoM.kicad_sch)

Commit message: Working on schematic
Other:
- sheet 100- Connectors renamed 200- Connectors
- sheet 100- PSoM ports: added +3V3, CE, LED_MOSI, PL, SPI_CLK, SPI_MISO, VSYS; removed none
Changed lines of the file:
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@@
     (stroke (width 0.1524) (type solid))
     (fill (color 0 0 0 0.0000))
-    (property "Sheetname" "100- Connectors" (at 167.64 24.3234 0)
+    (property "Sheetname" "200- Connectors" (at 167.64 24.3234 0)
       (effects (font (size 2 2)) (justify left bottom))
     )
@@
       (effects (font (size 1.27 1.27)) (justify right))
     )
-    (pin "D-" bidirectional (at 62.23 71.12 270)
-      (effects (font (size 1.27 1.27)) (justify left))
+    (pin "D-" bidirectional (at 83.82 43.18 0)
+      (effects (font (size 1.27 1.27)) (justify right))
     )
-    (pin "D+" bidirectional (at 58.42 71.12 270)
-      (effects (font (size 1.27 1.27)) (justify left))
+    (pin "D+" bidirectional (at 83.82 40.64 0)
+      (effects (font (size 1.27 1.27)) (justify right))
     )
     (pin "GND" passive (at 69.85 71.12 270)
@@
       (effects (font (size 1.27 1.27)) (justify right))
     )
+    (pin "SPI_MISO" output (at 83.82 53.34 0)
+      (effects (font (size 1.27 1.27)) (justify right))
+    )
+    (pin "SPI_CLK" input (at 83.82 55.88 0)
+      (effects (font (size 1.27 1.27)) (justify right))
+    )
+    (pin "LED_MOSI" input (at 83.82 68.58 0)
+      (effects (font (size 1.27 1.27)) (justify right))
+    )
+    (pin "PL" input (at 83.82 60.96 0)
+      (effects (font (size 1.27 1.27)) (justify right))
+    )
+    (pin "CE" input (at 83.82 58.42 0)
+      (effects (font (size 1.27 1.27)) (justify right))
+    )
+    (pin "+3V3" input (at 83.82 25.4 0)
+      (effects (font (size 1.27 1.27)) (justify right))
+    )
+    (pin "VSYS" input (at 83.82 30.48 0)
+      (effects (font (size 1.27 1.27)) (justify right))
+    )
     (instances
       (project "PMK_Keyboard_HW01"
-        (path "/c3b08055-08a5-4979-9bf8-f36ab0917722" (page "3"))
+        (path "/c3b08055-08a5-4979-9bf8-f36ab0917722" (page "1"))
       )
     )

Commit message: Started routing
Other:
- sheet 500- Shift Register - Switch renamed 300- Shift Register - Switch
- sheet 600- LEDs renamed 400- LEDs
- sheet 100- PSoM ports: added INT, SCL, SDA, SPI_MOSI; removed none
- sheet 200- Connectors ports: added 3V3, INT, MISO, MOSI, NCS, SCL, SCLK, SDA; removed none
- sheet 400- LEDs ports: added VSYS; removed VDD

Commit message: working on routing
Other:
- sheet 100- PSoM ports: added A, B; removed none
- sheet 300- Shift Register - Switch ports: added A, B; removed none

Commit message: Need to add some silkscreenthen done!
Other:
- sheet 100- PSoM ports: added GP_CE; removed none
- sheet 200- Connectors ports: added GP_CE; removed none
Changed lines of the file:
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@@
+    (stroke (width 0) (type default))
+  )
+  (wire (pts (xy 119.38 71.12) (xy 162.56 71.12))
     (stroke (width 0) (type default))
   )
@@
       (effects (font (size 1.27 1.27)) (justify right))
     )
+    (pin "GP_CE" input (at 162.56 71.12 180)
+      (effects (font (size 1.27 1.27)) (justify left))
+    )
     (instances
       (project "PMK_Keyboard_HW01"
@@
       (effects (font (size 1.27 1.27)) (justify right))
     )
+    (pin "GP_CE" input (at 119.38 71.12 0)
+      (effects (font (size 1.27 1.27)) (justify right))
+    )

Commit message: added mounting holes + fix in ref des
Other:
- sheet 100- PSoM renamed 200- PSoM
- sheet 200- Connectors renamed 300- Connectors
- sheet 300- Shift Register - Switch renamed 400- Shift Register - Switch
- sheet 400- LEDs renamed 500- LEDs
Changed lines of the file:
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@@
   (symbol (lib_id "power:+3V3") (at 210.82 30.48 0) (unit 1)
     (in_bom yes) (on_board yes) (dnp no) (fields_autoplaced)
-    (property "Reference" "#PWR0102" (at 210.82 34.29 0)
+    (property "Reference" "#PWR0302" (at 210.82 34.29 0)
       (effects (font (size 1.27 1.27)) hide)
     )
@@
       (project "PMK_Keyboard_HW01"
         (path "/c3b08055-08a5-4979-9bf8-f36ab0917722"
-          (reference "#PWR0102") (unit 1)
+          (reference "#PWR0302") (unit 1)
         )
       )
@@
   (symbol (lib_id "power:+3V3") (at 96.52 30.48 0) (unit 1)
     (in_bom yes) (on_board yes) (dnp no) (fields_autoplaced)
-    (property "Reference" "#PWR0101" (at 96.52 34.29 0)
+    (property "Reference" "#PWR0301" (at 96.52 34.29 0)
       (effects (font (size 1.27 1.27)) hide)
     )
@@
       (project "PMK_Keyboard_HW01"
         (path "/c3b08055-08a5-4979-9bf8-f36ab0917722"
-          (reference "#PWR0101") (unit 1)
+          (reference "#PWR0301") (unit 1)
         )
       )
@@
   (symbol (lib_id "power:+3V3") (at 104.14 99.06 0) (unit 1)
     (in_bom yes) (on_board yes) (dnp no) (fields_autoplaced)
-    (property "Reference" "#PWR0105" (at 104.14 102.87 0)
+    (property "Reference" "#PWR0305" (at 104.14 102.87 0)
       (effects (font (size 1.27 1.27)) hide)
     )
@@
       (project "PMK_Keyboard_HW01"
         (path "/c3b08055-08a5-4979-9bf8-f36ab0917722"
-          (reference "#PWR0105") (unit 1)
+          (reference "#PWR0305") (unit 1)
         )
       )
@@
   (symbol (lib_id "power:GND") (at 104.14 154.94 0) (unit 1)
     (in_bom yes) (on_board yes) (dnp no) (fields_autoplaced)
-    (property "Reference" "#PWR0106" (at 104.14 161.29 0)
+    (property "Reference" "#PWR0306" (at 104.14 161.29 0)
       (effects (font (size 1.27 1.27)) hide)
     )
@@
       (project "PMK_Keyboard_HW01"
         (path "/c3b08055-08a5-4979-9bf8-f36ab0917722"
-          (reference "#PWR0106") (unit 1)
+          (reference "#PWR0306") (unit 1)
         )
       )
@@
   (symbol (lib_id "power:GND") (at 215.9 154.94 0) (unit 1)
     (in_bom yes) (on_board yes) (dnp no) (fields_autoplaced)
-    (property "Reference" "#PWR0107" (at 215.9 161.29 0)
+    (property "Reference" "#PWR0307" (at 215.9 161.29 0)
       (effects (font (size 1.27 1.27)) hide)
     )
@@
       (project "PMK_Keyboard_HW01"
         (path "/c3b08055-08a5-4979-9bf8-f36ab0917722"
-          (reference "#PWR0107") (unit 1)
+          (reference "#PWR0307") (unit 1)
         )
       )
@@
   (symbol (lib_id "power:GND") (at 104.14 86.36 0) (unit 1)
     (in_bom yes) (on_board yes) (dnp no) (fields_autoplaced)
-    (property "Reference" "#PWR0103" (at 104.14 92.71 0)
+    (property "Reference" "#PWR0303" (at 104.14 92.71 0)
       (effects (font (size 1.27 1.27)) hide)
     )
@@
       (project "PMK_Keyboard_HW01"
         (path "/c3b08055-08a5-4979-9bf8-f36ab0917722"
-          (reference "#PWR0103") (unit 1)
+          (reference "#PWR0303") (unit 1)
         )
       )
@@
   (symbol (lib_id "power:GND") (at 215.9 86.36 0) (unit 1)
     (in_bom yes) (on_board yes) (dnp no) (fields_autoplaced)
-    (property "Reference" "#PWR0104" (at 215.9 92.71 0)
+    (property "Reference" "#PWR0304" (at 215.9 92.71 0)
       (effects (font (size 1.27 1.27)) hide)
     )
@@
       (project "PMK_Keyboard_HW01"
         (path "/c3b08055-08a5-4979-9bf8-f36ab0917722"
-          (reference "#PWR0104") (unit 1)
+          (reference "#PWR0304") (unit 1)
         )
       )
@@
     (stroke (width 0.1524) (type solid))
     (fill (color 0 0 0 0.0000))
-    (property "Sheetname" "300- Shift Register - Switch" (at 55.88 100.5234 0)
+    (property "Sheetname" "400- Shift Register - Switch" (at 55.88 100.5234 0)
       (effects (font (size 2 2)) (justify left bottom))
     )
@@
     (stroke (width 0.1524) (type solid))
     (fill (color 0 0 0 0.0000))
-    (property "Sheetname" "200- Connectors" (at 162.56 31.9434 0)
+    (property "Sheetname" "300- Connectors" (at 162.56 31.9434 0)
       (effects (font (size 2 2)) (justify left bottom))
     )
@@
     (stroke (width 0.1524) (type solid))
     (fill (color 0 0 0 0.0000))
-    (property "Sheetname" "400- LEDs" (at 162.56 100.5234 0)
+    (property "Sheetname" "500- LEDs" (at 162.56 100.5234 0)
       (effects (font (size 2 2)) (justify left bottom))
     )
@@
     (stroke (width 0.1524) (type solid))
     (fill (color 0 0 0 0.0000))
-    (property "Sheetname" "100- PSoM" (at 55.88 31.9434 0)
-      (effects (font (size 2 2)) (justify left bottom))
-    )
+    (property "Sheetname" "200- PSoM" (at 55.88 31.9434 0)
+      (effects (font (size 2 2)) (justify left bottom))
+    )
