File: Hardware/PMK_Keyboard/PMK_Keyboard_02.kicad_pro/PMK_Keyboard_02.kicad_pro.kicad_pcb (KiCad board)
At the start: 2 copper layers, 145 x 111.8 mm, 88 parts, among them J201 PSoM_ESP32S2_Carrier_Board, J202 PSoM_ESP32S2_Carrier_Board, J303 USB4510-03-1-A, J304 Conn_01x05_Pin, J305 505110-1292, J306 S2B-PH-SM4-TB, SW301 450405020524, SW401 SW_Push, SW402 SW_Push, SW403 SW_Push, SW404 SW_Push, SW405 SW_Push, SW406 SW_Push, SW407 SW_Push, SW408 SW_Push, SW409 SW_Push, SW410 SW_Push, SW411 SW_Push, SW412 SW_Push, SW413 SW_Push, SW414 SW_Push, SW415 SW_Push, SW416 SW_Push, SW417 SW_Push, SW418 SW_Push, SW419 SW_Push, SW420 SW_Push, SW421 SW_Push, SW422 SW_Push, SW423 SW_Push, SW424 SW_Push, SW425 SW_Push, SW426 SW_Push, SW427 SW_Push, SW428 SW_Push, SW429 SW_Push, SW430 RIC11-22S10D5S-TH, U401 SN74HC165PWR, U402 SN74HC165PWR, U403 SN74HC165PWR, U404 SN74HC165PWR

Commit message: added module connector
Parts:
- added D530: YF923_2020_WS2812_LED, Component_lib:YF923_2020_WS2812_LED_DUALSIDE, F.Cu at (209.5, 118.0)
- added U405: SN74LVC2G04DBVRG4, Component_lib:SOP95P280X145-6N, F.Cu at (211.5, 137.0)
- renumbered J303 to J301, J306 to J303
Connections:
- D529 pad 4: unconnected-(D529-DO-Pad4) -> Net-(D529-DO)
- J201 pad 25: /200- PSoM/SDA -> /200- PSoM/GP_CE
- J202 pad 25: /200- PSoM/SDA -> /200- PSoM/GP_CE
Routing:
- net unconnected-(D529-DO-Pad4): track 3.31 -> 0.00 mm, vias 1 -> 0
- net Net-(D529-DO): track 0.00 -> 3.31 mm, vias 0 -> 1
- net /200- PSoM/SDA: vias 2 -> 0
- net /200- PSoM/GP_CE: vias 2 -> 4
