File: Hardware/PMK_Keyboard/PMK_Keyboard_02.kicad_pro/PMK_Keyboard_02.kicad_pro.kicad_pcb (KiCad board)
At the start: 2 copper layers, 145 x 111.8 mm, 101 parts, among them J201 PSoM_ESP32S2_Carrier_Board, J202 PSoM_ESP32S2_Carrier_Board, J301 USB4510-03-1-A, J302 Conn_01x02, J303 S2B-PH-SM4-TB, J304 FH12-12S-0.5SH_55_, SW301 450405020524, SW401 SW_Push, SW402 SW_Push, SW403 SW_Push, SW404 SW_Push, SW405 SW_Push, SW406 SW_Push, SW407 SW_Push, SW408 SW_Push, SW409 SW_Push, SW410 SW_Push, SW411 SW_Push, SW412 SW_Push, SW413 SW_Push, SW414 SW_Push, SW415 SW_Push, SW416 SW_Push, SW417 SW_Push, SW418 SW_Push, SW419 SW_Push, SW420 SW_Push, SW421 SW_Push, SW422 SW_Push, SW423 SW_Push, SW424 SW_Push, SW425 SW_Push, SW426 SW_Push, SW427 SW_Push, SW428 SW_Push, SW429 SW_Push, SW430 RIC11-22S10D5S-TH, U401 SN74HC165PWR, U402 SN74HC165PWR, U403 SN74HC165PWR, U404 SN74HC165PWR, U405 SN74LVC2G04DBVRG4

Commit message: routing almost done
Parts:
- moved TP204 43.1 mm to (201.8, 98.8)
- moved TP207 41.9 mm to (218.0, 59.6)
- moved TP206 41.3 mm to (216.2, 57.8)
- moved TP201 39.4 mm to (201.8, 94.0)
- moved TP202 38.2 mm to (201.8, 96.4)
- moved TP205 37.6 mm to (201.8, 91.6)
- moved TP203 36.3 mm to (201.8, 89.2)
- moved TP208 36.3 mm to (201.8, 86.8)
Connections:
- D525 pad 3: Net-(D524-DO) -> Net-(D525-DIN)
- D529 pad 4: Net-(D529-DO) -> unconnected-(D529-DO-Pad4)
- D530 pad 3: Net-(D529-DO) -> Net-(D524-DO)
- D530 pad 4: unconnected-(D530-DO-Pad4) -> Net-(D525-DIN)
- J201 pad 31: /200- PSoM/DB_A -> /200- PSoM/DB_B
- J201 pad 33: /200- PSoM/DB_B -> /200- PSoM/DB_A
- J202 pad 31: /200- PSoM/DB_A -> /200- PSoM/DB_B
- J202 pad 33: /200- PSoM/DB_B -> /200- PSoM/DB_A
Routing:
- net /200- PSoM/SR_CE: track 21.4 -> 126.7 mm, vias 2 -> 8
- net /200- PSoM/DB_A: track 4.55 -> 108.2 mm, vias 0 -> 1
- net /200- PSoM/DB_B: track 4.34 -> 99.9 mm, vias 0 -> 1
- net /200- PSoM/PL: track 13.0 -> 90.1 mm, vias 3 -> 8
- net Net-(D525-DIN): track 0.00 -> 46.6 mm, vias 0 -> 2
- net /200- PSoM/SDA: track 39.4 -> 82.4 mm
- net VDD: track 732.4 -> 769.8 mm, vias 31 -> 36
- net /200- PSoM/SPI_CLK_ESP: track 3.45 -> 27.5 mm, vias 0 -> 5
- net /200- PSoM/TX: track 0.00 -> 24.0 mm, vias 0 -> 3
- net /200- PSoM/SCL: track 40.3 -> 64.2 mm
- net /200- PSoM/RX: track 0.00 -> 23.7 mm, vias 0 -> 3
- net /200- PSoM/SPI_MISO: track 54.9 -> 74.2 mm, vias 4 -> 6
- net /200- PSoM/GPIO3: track 39.3 -> 58.2 mm, vias 0 -> 1
- net /200- PSoM/GPIO2: track 38.6 -> 56.1 mm, vias 0 -> 1
- net /200- PSoM/SPI_CLK: track 91.6 -> 74.4 mm, vias 3 -> 2
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
Commit message: PMK_Keyboard_02 is done
Parts:
- added J305: FFC2B28-12-G, Component_lib:GCT_FFC2B28-12-G, B.Cu at (207.3, 105.0)
- J304: value FH12-12S-0.5SH_55_ -> FFC2B28-12-G; footprint Component_lib:FH12-12S-0.5SH_55_ -> Component_lib:GCT_FFC2B28-12-G
- moved J304 2.37 mm to (207.3, 105.0)
- moved U403 1.50 mm to (198.0, 115.0)
- moved U401 1.50 mm to (198.0, 77.0)
- moved U402 1.50 mm to (198.0, 96.5)
- moved U404 1.50 mm to (198.0, 134.8)
- moved RN402 0.80 mm to (200.6, 96.5)
- moved RN401 0.80 mm to (200.6, 77.0)
- moved TP201 0.60 mm to (202.4, 94.0)
- moved TP202 0.60 mm to (202.4, 96.4)
- moved TP203 0.60 mm to (202.4, 89.2)
- moved TP204 0.60 mm to (202.4, 98.8)
- moved TP205 0.60 mm to (202.4, 91.6)
- moved TP208 0.60 mm to (202.4, 86.8)
Routing:
- net /200- PSoM/GPIO3: track 58.2 -> 82.2 mm, vias 1 -> 4
- net /200- PSoM/GPIO2: track 56.1 -> 78.3 mm, vias 1 -> 4
- net /200- PSoM/SPI_CLK: track 74.4 -> 91.0 mm, vias 2 -> 1
- net +3V3: track 126.3 -> 142.0 mm
- net /200- PSoM/SPI_MISO: track 74.2 -> 88.2 mm, vias 6 -> 7
- net /200- PSoM/SDA: track 82.4 -> 72.3 mm, vias 2 -> 5
- net GND: track 70.8 -> 80.9 mm, vias 192 -> 201
- net /200- PSoM/GP_CE: track 51.9 -> 61.0 mm, vias 1 -> 3
- net /200- PSoM/DR: track 51.0 -> 59.8 mm, vias 1 -> 2
- net /200- PSoM/SPI_MOSI: track 51.7 -> 60.5 mm, vias 3 -> 6
- net /200- PSoM/SCL: track 64.2 -> 71.3 mm
- net /200- PSoM/PL: track 90.1 -> 96.5 mm
- net /200- PSoM/DB_A: track 108.2 -> 111.2 mm
- net /200- PSoM/DB_B: track 99.9 -> 102.8 mm
- net /400- Shift Register - Switch/2-3: track 20.5 -> 23.3 mm
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Other:
- board text added: "PMK_HW02 inspired from Sofle"

Commit message: fixed typo on silkscreen, no new rev for this fix
Other:
- board text removed: "PMK_HW01 inspired from Sofle"
Changed lines of the file:
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@@
 		(layer "Edge.Cuts")
 	)
-	(gr_text "PMK_HW01 inspired from Sofle"
+	(gr_text "PMK_HW02 inspired from Sofle"
 		(at 118.1 146.4 340)
 		(layer "B.SilkS")
