File: Hardware/PMK_Keyboard/PMK_Keyboard_02.kicad_pro/ShiftRegisterSwitch.kicad_sch (KiCad schematic)
At the start: 41 parts, among them SW401 SW_Push, SW402 SW_Push, SW403 SW_Push, SW404 SW_Push, SW405 SW_Push, SW406 SW_Push, SW407 SW_Push, SW408 SW_Push, SW409 SW_Push, SW410 SW_Push, SW411 SW_Push, SW412 SW_Push, SW413 SW_Push, SW414 SW_Push, SW415 SW_Push, SW416 SW_Push, SW417 SW_Push, SW418 SW_Push, SW419 SW_Push, SW420 SW_Push, SW421 SW_Push, SW422 SW_Push, SW423 SW_Push, SW424 SW_Push, SW425 SW_Push, SW426 SW_Push, SW427 SW_Push, SW428 SW_Push, SW429 SW_Push, SW430 RIC11-22S10D5S-TH, U201 SN74LVC3G04DCTR, U401 SN74HC165PWR, U402 SN74HC165PWR, U403 SN74HC165PWR, U404 SN74HC165PWR

Commit message: working on schematic 02
Parts:
- removed U201: SN74LVC3G04DCTR, SOP65P400X130-8N, symbol Component_lib:SN74LVC3G04DCTR
- added C401, C402: 10n, symbol Component_lib:C
- added C403: 100n, symbol Component_lib:C
- added R401, R402, R403, R404: 10k, symbol Component_lib:R
- added U405: SN74LVC2G04DBVRG4, SOP95P280X145-6N, symbol Component_lib:SN74LVC2G04DBVRG4
- renumbered R401 to R405, R402 to R406
Connections:
- net +3V3: now also C403.1, R401.2, R403.2, U405.5 (VCC)
- net A: now also R401.1, R402.2, U405.6 (1Y)
- net B: now also R403.1, R404.2, U405.4 (2Y)
- net GND: now also C401.2, C402.2, C403.2, U405.2 (GND)
- new net F_A: C401.1, R402.1, U405.1 (1A)
- new net F_B: C402.1, R404.1, U405.3 (2A)
Other:
- moved on the sheet: R405, R406, SW430

Commit message: Schematic 02 done
Parts:
- C401, C402, C403: footprint (none) -> Capacitor_SMD:C_0402_1005Metric
- R401, R402, R403, R404: footprint (none) -> Resistor_SMD:R_0201_0603Metric
- R405, R406: footprint (none) -> Resistor_SMD:R_0402_1005Metric
- U405: footprint SOP95P280X145-6N -> Component_lib:SOP95P280X145-6N
Changed lines of the file:
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@@
 			)
 		)
-		(property "Footprint" ""
+		(property "Footprint" "Capacitor_SMD:C_0402_1005Metric"
 			(at 359.7148 160.02 0)
 			(effects
@@
 			)
 		)
-		(property "Footprint" ""
+		(property "Footprint" "Resistor_SMD:R_0402_1005Metric"
 			(at 372.11 194.818 90)
 			(effects
@@
 			)
 		)
-		(property "Footprint" ""
+		(property "Footprint" "Capacitor_SMD:C_0402_1005Metric"
 			(at 341.9348 193.04 0)
 			(effects
@@
 			)
 		)
-		(property "Footprint" ""
+		(property "Footprint" "Resistor_SMD:R_0201_0603Metric"
 			(at 384.81 151.638 90)
 			(effects
@@
 			)
 		)
-		(property "Footprint" ""
+		(property "Footprint" "Resistor_SMD:R_0201_0603Metric"
 			(at 354.33 151.638 90)
 			(effects
@@
 			)
 		)
-		(property "Footprint" ""
+		(property "Footprint" "Capacitor_SMD:C_0402_1005Metric"
 			(at 390.1948 160.02 0)
 			(effects
@@
 			)
 		)
-		(property "Footprint" "SOP95P280X145-6N"
+		(property "Footprint" "Component_lib:SOP95P280X145-6N"
 			(at 326.39 280.34 0)
 			(effects
@@
 			)
 		)
-		(property "Footprint" ""
+		(property "Footprint" "Resistor_SMD:R_0201_0603Metric"
 			(at 346.202 143.51 90)
 			(effects
@@
 			)
 		)
-		(property "Footprint" ""
+		(property "Footprint" "Resistor_SMD:R_0201_0603Metric"
 			(at 376.682 143.51 90)
 			(effects
@@
 			)
 		)
-		(property "Footprint" ""
+		(property "Footprint" "Resistor_SMD:R_0402_1005Metric"
 			(at 372.11 184.658 90)
 			(effects

Commit message: working on routing
Connections:
- net 30: now also R405.2; no longer SW430.S2
- net 31: now also R406.2; no longer R405.2
- net 32: now also SW430.S2; no longer R406.2
- net A: no longer R405.1, U405.6 (1Y)
- net B: no longer R406.1, U405.4 (2Y)
- new net DB_A: R405.1, U405.6 (1Y)
- new net DB_B: R406.1, U405.4 (2Y)
Changed lines of the file:
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@@
 		)
 	)
-	(label "31"
+	(label "30"
 		(at 378.46 182.88 0)
 		(fields_autoplaced yes)
@@
 		)
 	)
-	(label "30"
+	(label "32"
 		(at 327.66 149.86 0)
 		(fields_autoplaced yes)
@@
 		)
 	)
-	(label "32"
+	(label "31"
 		(at 378.46 193.04 0)
 		(fields_autoplaced yes)
@@
 		)
 	)
-	(hierarchical_label "B"
+	(hierarchical_label "DB_B"
 		(shape output)
 		(at 386.08 63.5 0)
@@
 		)
 	)
-	(hierarchical_label "A"
+	(hierarchical_label "DB_A"
 		(shape output)
 		(at 386.08 58.42 0)

Commit message: updated key switch to kailh v2
Parts:
- SW401, SW402, SW403, SW404, SW405, SW406, SW407, SW408, SW409, SW410, SW411, SW412, SW413, SW414, SW415, SW416, SW417, SW418, SW419, SW420, SW421, SW422, SW423, SW424, SW425, SW426, SW427, SW428, SW429: footprint Component_lib:Kailh_socket_PG1350_reversible -> Component_lib:Kailh_socket_PG1350_reversible_V1V2
Changed lines of the file:
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@@
 			)
 		)
-		(property "Footprint" "Component_lib:Kailh_socket_PG1350_reversible"
+		(property "Footprint" "Component_lib:Kailh_socket_PG1350_reversible_V1V2"
 			(at 68.58 200.66 0)
 			(effects
@@
 			)
 		)
-		(property "Footprint" "Component_lib:Kailh_socket_PG1350_reversible"
+		(property "Footprint" "Component_lib:Kailh_socket_PG1350_reversible_V1V2"
 			(at 63.5 200.66 0)
 			(effects
@@
 			)
 		)
-		(property "Footprint" "Component_lib:Kailh_socket_PG1350_reversible"
+		(property "Footprint" "Component_lib:Kailh_socket_PG1350_reversible_V1V2"
 			(at 83.82 200.66 0)
 			(effects
@@
 			)
 		)
-		(property "Footprint" "Component_lib:Kailh_socket_PG1350_reversible"
+		(property "Footprint" "Component_lib:Kailh_socket_PG1350_reversible_V1V2"
 			(at 93.98 200.66 0)
 			(effects
@@
 			)
 		)
-		(property "Footprint" "Component_lib:Kailh_socket_PG1350_reversible"
+		(property "Footprint" "Component_lib:Kailh_socket_PG1350_reversible_V1V2"
 			(at 58.42 200.66 0)
 			(effects
@@
 			)
 		)
-		(property "Footprint" "Component_lib:Kailh_socket_PG1350_reversible"
+		(property "Footprint" "Component_lib:Kailh_socket_PG1350_reversible_V1V2"
 			(at 210.82 200.66 0)
 			(effects
@@
 			)
 		)
-		(property "Footprint" "Component_lib:Kailh_socket_PG1350_reversible"
+		(property "Footprint" "Component_lib:Kailh_socket_PG1350_reversible_V1V2"
 			(at 121.92 200.66 0)
 			(effects
@@
 			)
 		)
-		(property "Footprint" "Component_lib:Kailh_socket_PG1350_reversible"
+		(property "Footprint" "Component_lib:Kailh_socket_PG1350_reversible_V1V2"
 			(at 137.16 200.66 0)
 			(effects
@@
 			)
 		)
-		(property "Footprint" "Component_lib:Kailh_socket_PG1350_reversible"
+		(property "Footprint" "Component_lib:Kailh_socket_PG1350_reversible_V1V2"
 			(at 205.74 200.66 0)
 			(effects
@@
 			)
 		)
-		(property "Footprint" "Component_lib:Kailh_socket_PG1350_reversible"
+		(property "Footprint" "Component_lib:Kailh_socket_PG1350_reversible_V1V2"
 			(at 220.98 200.66 0)
 			(effects
@@
 			)
 		)
-		(property "Footprint" "Component_lib:Kailh_socket_PG1350_reversible"
+		(property "Footprint" "Component_lib:Kailh_socket_PG1350_reversible_V1V2"
 			(at 264.16 200.66 0)
 			(effects
@@
 			)
 		)
-		(property "Footprint" "Component_lib:Kailh_socket_PG1350_reversible"
+		(property "Footprint" "Component_lib:Kailh_socket_PG1350_reversible_V1V2"
 			(at 88.9 200.66 0)
 			(effects
@@
 			)
 		)
-		(property "Footprint" "Component_lib:Kailh_socket_PG1350_reversible"
+		(property "Footprint" "Component_lib:Kailh_socket_PG1350_reversible_V1V2"
 			(at 185.42 200.66 0)
 			(effects
@@
 			)
 		)
-		(property "Footprint" "Component_lib:Kailh_socket_PG1350_reversible"
+		(property "Footprint" "Component_lib:Kailh_socket_PG1350_reversible_V1V2"
 			(at 195.58 200.66 0)
 			(effects
@@
 			)
 		)
-		(property "Footprint" "Component_lib:Kailh_socket_PG1350_reversible"
+		(property "Footprint" "Component_lib:Kailh_socket_PG1350_reversible_V1V2"
 			(at 157.48 200.66 0)
 			(effects
@@
 			)
 		)
-		(property "Footprint" "Component_lib:Kailh_socket_PG1350_reversible"
+		(property "Footprint" "Component_lib:Kailh_socket_PG1350_reversible_V1V2"
 			(at 254 200.66 0)
 			(effects
@@
 			)
 		)
-		(property "Footprint" "Component_lib:Kailh_socket_PG1350_reversible"
+		(property "Footprint" "Component_lib:Kailh_socket_PG1350_reversible_V1V2"
 			(at 269.24 200.66 0)
 			(effects
@@
 			)
 		)
-		(property "Footprint" "Component_lib:Kailh_socket_PG1350_reversible"
+		(property "Footprint" "Component_lib:Kailh_socket_PG1350_reversible_V1V2"
 			(at 200.66 200.66 0)
 			(effects
@@
 			)
 		)
-		(property "Footprint" "Component_lib:Kailh_socket_PG1350_reversible"
+		(property "Footprint" "Component_lib:Kailh_socket_PG1350_reversible_V1V2"
 			(at 259.08 200.66 0)
 			(effects
@@
 			)
 		)
-		(property "Footprint" "Component_lib:Kailh_socket_PG1350_reversible"
+		(property "Footprint" "Component_lib:Kailh_socket_PG1350_reversible_V1V2"
 			(at 127 200.66 0)
 			(effects
@@
 			)
 		)
-		(property "Footprint" "Component_lib:Kailh_socket_PG1350_reversible"
+		(property "Footprint" "Component_lib:Kailh_socket_PG1350_reversible_V1V2"
 			(at 78.74 200.66 0)
 			(effects
@@
 			)
 		)
-		(property "Footprint" "Component_lib:Kailh_socket_PG1350_reversible"
+		(property "Footprint" "Component_lib:Kailh_socket_PG1350_reversible_V1V2"
 			(at 152.4 200.66 0)
 			(effects
@@
 			)
 		)
-		(property "Footprint" "Component_lib:Kailh_socket_PG1350_reversible"
+		(property "Footprint" "Component_lib:Kailh_socket_PG1350_reversible_V1V2"
 			(at 190.5 200.66 0)
 			(effects
@@
 			)
 		)
-		(property "Footprint" "Component_lib:Kailh_socket_PG1350_reversible"
+		(property "Footprint" "Component_lib:Kailh_socket_PG1350_reversible_V1V2"
 			(at 215.9 200.66 0)
 			(effects
@@
 			)
 		)
-		(property "Footprint" "Component_lib:Kailh_socket_PG1350_reversible"
+		(property "Footprint" "Component_lib:Kailh_socket_PG1350_reversible_V1V2"
 			(at 132.08 200.66 0)
 			(effects
@@
 			)
 		)
-		(property "Footprint" "Component_lib:Kailh_socket_PG1350_reversible"
+		(property "Footprint" "Component_lib:Kailh_socket_PG1350_reversible_V1V2"
 			(at 142.24 200.66 0)
 			(effects
@@
 			)
 		)
-		(property "Footprint" "Component_lib:Kailh_socket_PG1350_reversible"
+		(property "Footprint" "Component_lib:Kailh_socket_PG1350_reversible_V1V2"
 			(at 147.32 200.66 0)
 			(effects
@@
 			)
 		)
-		(property "Footprint" "Component_lib:Kailh_socket_PG1350_reversible"
+		(property "Footprint" "Component_lib:Kailh_socket_PG1350_reversible_V1V2"
 			(at 248.92 200.66 0)
 			(effects
@@
 			)
 		)
-		(property "Footprint" "Component_lib:Kailh_socket_PG1350_reversible"
+		(property "Footprint" "Component_lib:Kailh_socket_PG1350_reversible_V1V2"
 			(at 73.66 200.66 0)
 			(effects
