File: Hardware/PMK_Keyboard/PMK_Keyboard_02.kicad_pro/LEDs.kicad_sch (KiCad schematic)
At the start: 30 parts

Commit message: routing almost done
Connections:
- net at D530.3 (DIN): now also D524.4 (DO); no longer D529.4 (DO)
- net at D530.4 (DO): now also D525.3 (DIN)
Other:
- moved on the sheet: D525, D526, D530
Changed lines of the file:
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@@
 	(wire
 		(pts
-			(xy 88.9 154.94) (xy 88.9 157.48)
+			(xy 231.14 116.84) (xy 231.14 119.38)
 		)
 		(stroke
@@
 	(wire
 		(pts
-			(xy 231.14 99.06) (xy 231.14 101.6)
+			(xy 248.92 99.06) (xy 248.92 101.6)
 		)
 		(stroke
@@
 	(wire
 		(pts
-			(xy 256.54 109.22) (xy 259.08 109.22)
+			(xy 274.32 109.22) (xy 276.86 109.22)
 		)
 		(stroke
@@
 	(wire
 		(pts
-			(xy 231.14 116.84) (xy 231.14 119.38)
+			(xy 248.92 116.84) (xy 248.92 119.38)
 		)
 		(stroke
@@
 	(wire
 		(pts
-			(xy 238.76 109.22) (xy 241.3 109.22)
+			(xy 256.54 109.22) (xy 259.08 109.22)
 		)
 		(stroke
@@
 	(wire
 		(pts
-			(xy 78.74 147.32) (xy 81.28 147.32)
+			(xy 238.76 109.22) (xy 241.3 109.22)
 		)
 		(stroke
@@
 	(wire
 		(pts
-			(xy 248.92 116.84) (xy 248.92 119.38)
+			(xy 266.7 116.84) (xy 266.7 119.38)
 		)
 		(stroke
@@
 	(wire
 		(pts
-			(xy 248.92 99.06) (xy 248.92 101.6)
+			(xy 266.7 99.06) (xy 266.7 101.6)
 		)
 		(stroke
@@
 	(wire
 		(pts
-			(xy 88.9 137.16) (xy 88.9 139.7)
+			(xy 231.14 99.06) (xy 231.14 101.6)
 		)
 		(stroke
@@
 	)
 	(label "LED_26_27"
-		(at 259.08 109.22 0)
+		(at 276.86 109.22 0)
 		(fields_autoplaced yes)
 		(effects
@@
 	(symbol
 		(lib_id "Component lib:YF923_2020_WS2812_LED")
-		(at 248.92 109.22 0)
+		(at 266.7 109.22 0)
 		(unit 1)
 		(exclude_from_sim no)
@@
 		(dnp no)
 		(property "Reference" "D526"
-			(at 254 101.6 0)
+			(at 271.78 101.6 0)
 			(effects
 				(font
@@
 		)
 		(property "Value" "YF923_2020_WS2812_LED"
-			(at 248.92 96.52 0)
+			(at 266.7 96.52 0)
 			(effects
 				(font
@@
 		)
 		(property "Footprint" "Component_lib:YF923_2020_WS2812_LED_DUALSIDE"
-			(at 250.19 116.84 0)
+			(at 267.97 116.84 0)
 			(effects
 				(font
@@
 		)
 		(property "Datasheet" "https://fr.aliexpress.com/item/4000770210584.html?spm=a2g0o.order_list.order_list_main.4.702f5e5bJqEWkF&gatewayAdapt=glo2fra"
-			(at 251.46 118.745 0)
+			(at 269.24 118.745 0)
 			(effects
 				(font
@@
 		)
 		(property "Description" ""
-			(at 248.92 109.22 0)
+			(at 266.7 109.22 0)
 			(effects
 				(font
@@
 	(symbol
 		(lib_id "Component lib:YF923_2020_WS2812_LED")
-		(at 88.9 147.32 0)
+		(at 231.14 109.22 0)
 		(unit 1)
 		(exclude_from_sim no)
@@
 		(dnp no)
 		(property "Reference" "D530"
-			(at 93.98 139.7 0)
+			(at 236.22 101.6 0)
 			(effects
 				(font
@@
 		)
 		(property "Value" "YF923_2020_WS2812_LED"
-			(at 88.9 134.62 0)
+			(at 231.14 96.52 0)
 			(effects
 				(font
@@
 		)
 		(property "Footprint" "Component_lib:YF923_2020_WS2812_LED_DUALSIDE"
-			(at 90.17 154.94 0)
+			(at 232.41 116.84 0)
 			(effects
 				(font
@@
 		)
 		(property "Datasheet" "https://fr.aliexpress.com/item/4000770210584.html?spm=a2g0o.order_list.order_list_main.4.702f5e5bJqEWkF&gatewayAdapt=glo2fra"
-			(at 91.44 156.845 0)
+			(at 233.68 118.745 0)
 			(effects
 				(font
@@
 		)
 		(property "Description" ""
-			(at 88.9 147.32 0)
+			(at 231.14 109.22 0)
 			(effects
 				(font
@@
 	(symbol
 		(lib_id "power:VDD")
-		(at 88.9 137.16 0)
+		(at 231.14 99.06 0)
 		(unit 1)
 		(exclude_from_sim no)
@@
 		(fields_autoplaced yes)
 		(property "Reference" "#PWR0209"
-			(at 88.9 140.97 0)
+			(at 231.14 102.87 0)
 			(effects
 				(font
@@
 		)
 		(property "Value" "VDD"
-			(at 88.9 133.5842 0)
+			(at 231.14 95.4842 0)
 			(effects
 				(font
@@
 		)
 		(property "Footprint" ""
-			(at 88.9 137.16 0)
+			(at 231.14 99.06 0)
 			(effects
 				(font
@@
 		)
 		(property "Datasheet" ""
-			(at 88.9 137.16 0)
+			(at 231.14 99.06 0)
 			(effects
 				(font
@@
 		)
 		(property "Description" ""
-			(at 88.9 137.16 0)
+			(at 231.14 99.06 0)
 			(effects
 				(font
@@
 	(symbol
 		(lib_id "power:GND")
-		(at 248.92 119.38 0)
+		(at 266.7 119.38 0)
 		(unit 1)
 		(exclude_from_sim no)
@@
 		(fields_autoplaced yes)
 		(property "Reference" "#PWR0554"
-			(at 248.92 125.73 0)
+			(at 266.7 125.73 0)
 			(effects
 				(font
@@
 		)
 		(property "Value" "GND"
-			(at 248.92 123.8234 0)
+			(at 266.7 123.8234 0)
 			(effects
 				(font
@@
 		)
 		(property "Footprint" ""
-			(at 248.92 119.38 0)
+			(at 266.7 119.38 0)
 			(effects
 				(font
@@
 		)
 		(property "Datasheet" ""
-			(at 248.92 119.38 0)
+			(at 266.7 119.38 0)
 			(effects
 				(font
@@
 		)
 		(property "Description" ""
-			(at 248.92 119.38 0)
+			(at 266.7 119.38 0)
 			(effects
 				(font
@@
 	(symbol
 		(lib_id "power:GND")
-		(at 231.14 119.38 0)
+		(at 248.92 119.38 0)
 		(unit 1)
 		(exclude_from_sim no)
@@
 		(fields_autoplaced yes)
 		(property "Reference" "#PWR0553"
-			(at 231.14 125.73 0)
+			(at 248.92 125.73 0)
 			(effects
 				(font
@@
 		)
 		(property "Value" "GND"
-			(at 231.14 123.8234 0)
+			(at 248.92 123.8234 0)
 			(effects
 				(font
@@
 		)
 		(property "Footprint" ""
-			(at 231.14 119.38 0)
+			(at 248.92 119.38 0)
 			(effects
 				(font
@@
 		)
 		(property "Datasheet" ""
-			(at 231.14 119.38 0)
+			(at 248.92 119.38 0)
 			(effects
 				(font
@@
 		)
 		(property "Description" ""
-			(at 231.14 119.38 0)
+			(at 248.92 119.38 0)
 			(effects
 				(font
@@
 	(symbol
 		(lib_id "power:VDD")
-		(at 231.14 99.06 0)
+		(at 248.92 99.06 0)
 		(unit 1)
 		(exclude_from_sim no)
@@
 		(fields_autoplaced yes)
 		(property "Reference" "#PWR0540"
-			(at 231.14 102.87 0)
+			(at 248.92 102.87 0)
 			(effects
 				(font
@@
 		)
 		(property "Value" "VDD"
-			(at 231.14 95.4842 0)
+			(at 248.92 95.4842 0)
 			(effects
 				(font
@@
 		)
 		(property "Footprint" ""
-			(at 231.14 99.06 0)
+			(at 248.92 99.06 0)
 			(effects
 				(font
@@
 		)
 		(property "Datasheet" ""
-			(at 231.14 99.06 0)
+			(at 248.92 99.06 0)
 			(effects
 				(font
@@
 		)
 		(property "Description" ""
-			(at 231.14 99.06 0)
+			(at 248.92 99.06 0)
 			(effects
 				(font
@@
 	(symbol
 		(lib_id "power:GND")
-		(at 88.9 157.48 0)
+		(at 231.14 119.38 0)
 		(unit 1)
 		(exclude_from_sim no)
@@
 		(fields_autoplaced yes)
 		(property "Reference" "#PWR0210"
-			(at 88.9 163.83 0)
+			(at 231.14 125.73 0)
 			(effects
 				(font
@@
 		)
 		(property "Value" "GND"
-			(at 88.9 161.9234 0)
+			(at 231.14 123.8234 0)
 			(effects
 				(font
@@
 		)
 		(property "Footprint" ""
-			(at 88.9 157.48 0)
+			(at 231.14 119.38 0)
 			(effects
 				(font
@@
 		)
 		(property "Datasheet" ""
-			(at 88.9 157.48 0)
+			(at 231.14 119.38 0)
 			(effects
 				(font
@@
 		)
 		(property "Description" ""
-			(at 88.9 157.48 0)
+			(at 231.14 119.38 0)
 			(effects
 				(font
@@
 	(symbol
 		(lib_id "Component lib:YF923_2020_WS2812_LED")
-		(at 231.14 109.22 0)
+		(at 248.92 109.22 0)
 		(unit 1)
 		(exclude_from_sim no)
@@
 		(dnp no)
 		(property "Reference" "D525"
-			(at 236.22 101.6 0)
+			(at 254 101.6 0)
 			(effects
 				(font
@@
 		)
 		(property "Value" "YF923_2020_WS2812_LED"
-			(at 231.14 96.52 0)
+			(at 248.92 96.52 0)
 			(effects
 				(font
@@
 		)
 		(property "Footprint" "Component_lib:YF923_2020_WS2812_LED_DUALSIDE"
-			(at 232.41 116.84 0)
+			(at 250.19 116.84 0)
 			(effects
 				(font
@@
 		)
 		(property "Datasheet" "https://fr.aliexpress.com/item/4000770210584.html?spm=a2g0o.order_list.order_list_main.4.702f5e5bJqEWkF&gatewayAdapt=glo2fra"
-			(at 233.68 118.745 0)
+			(at 251.46 118.745 0)
 			(effects
 				(font
@@
 		)
 		(property "Description" ""
-			(at 231.14 109.22 0)
+			(at 248.92 109.22 0)
 			(effects
 				(font
@@
 	(symbol
 		(lib_id "power:VDD")
-		(at 248.92 99.06 0)
+		(at 266.7 99.06 0)
 		(unit 1)
 		(exclude_from_sim no)
@@
 		(fields_autoplaced yes)
 		(property "Reference" "#PWR0541"
-			(at 248.92 102.87 0)
+			(at 266.7 102.87 0)
 			(effects
 				(font
@@
 		)
 		(property "Value" "VDD"
-			(at 248.92 95.4842 0)
+			(at 266.7 95.4842 0)
 			(effects
 				(font
@@
 		)
 		(property "Footprint" ""
-			(at 248.92 99.06 0)
+			(at 266.7 99.06 0)
 			(effects
 				(font
@@
 		)
 		(property "Datasheet" ""
-			(at 248.92 99.06 0)
+			(at 266.7 99.06 0)
 			(effects
 				(font
@@
 		)
 		(property "Description" ""
-			(at 248.92 99.06 0)
+			(at 266.7 99.06 0)
 			(effects
 				(font
