File: Hardware/PMK_Keyboard/PMK_Keyboard_02.kicad_pro/Connectors.kicad_sch (KiCad schematic)
At the start: 8 parts, among them J301 USB4510-03-1-A, J302 Conn_01x02, J303 S2B-PH-SM4-TB, SW301 450405020524

Commit message: working on schematic 02
Changed lines of the file:
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@@
-	(wire
-		(pts
-			(xy 203.2 73.66) (xy 203.2 106.68)
-		)
-		(stroke
-			(width 0)
-			(type default)
-		)
-	)
 	(wire
 		(pts
@@
 	(wire
 		(pts
-			(xy 203.2 73.66) (xy 205.74 73.66)
-		)
-		(stroke
-			(width 0)
-			(type default)
-		)
-	)
-	(wire
-		(pts
 			(xy 50.8 111.76) (xy 50.8 109.22)
 		)
@@
 	(wire
 		(pts
-			(xy 200.66 78.74) (xy 205.74 78.74)
-		)
-		(stroke
-			(width 0)
-			(type default)
-		)
-	)
-	(wire
-		(pts
 			(xy 271.78 86.36) (xy 274.32 86.36)
 		)
@@
 	(wire
 		(pts
-			(xy 162.56 83.82) (xy 162.56 81.28)
-		)
-		(stroke
-			(width 0)
-			(type default)
-		)
-	)
-	(wire
-		(pts
 			(xy 271.78 66.04) (xy 274.32 66.04)
 		)
@@
 	(wire
 		(pts
-			(xy 162.56 81.28) (xy 165.1 81.28)
-		)
-		(stroke
-			(width 0)
-			(type default)
-		)
-	)
-	(wire
-		(pts
 			(xy 63.5 66.04) (xy 66.04 66.04)
 		)
@@
 		(pts
 			(xy 200.66 88.9) (xy 205.74 88.9)
-		)
-		(stroke
-			(width 0)
-			(type default)
-		)
-	)
-	(wire
-		(pts
-			(xy 200.66 76.2) (xy 205.74 76.2)
 		)
 		(stroke
@@
 		)
 	)
-	(label "SCL"
-		(at 200.66 78.74 180)
-		(fields_autoplaced yes)
-		(effects
-			(font
-				(size 1.27 1.27)
-			)
-			(justify right bottom)
-		)
-	)
 	(label "NCS"
 		(at 271.78 81.28 180)
@@
 	(label "BTN2"
 		(at 200.66 83.82 180)
-		(fields_autoplaced yes)
-		(effects
-			(font
-				(size 1.27 1.27)
-			)
-			(justify right bottom)
-		)
-	)
-	(label "SDA"
-		(at 200.66 76.2 180)
 		(fields_autoplaced yes)
 		(effects
@@
 	(symbol
 		(lib_id "power:GND")
-		(at 162.56 83.82 0)
+		(at 162.56 104.14 0)
 		(unit 1)
 		(exclude_from_sim no)
@@
 		(fields_autoplaced yes)
 		(property "Reference" "#PWR0320"
-			(at 162.56 90.17 0)
+			(at 162.56 110.49 0)
 			(effects
 				(font
@@
 		)
 		(property "Value" "GND"
-			(at 162.56 88.2634 0)
+			(at 162.56 108.5834 0)
 			(effects
 				(font
@@
 		)
 		(property "Footprint" ""
-			(at 162.56 83.82 0)
+			(at 162.56 104.14 0)
 			(effects
 				(font
@@
 		)
 		(property "Datasheet" ""
-			(at 162.56 83.82 0)
+			(at 162.56 104.14 0)
 			(effects
 				(font
@@
 		)
 		(property "Description" ""
-			(at 162.56 83.82 0)
+			(at 162.56 104.14 0)
 			(effects
 				(font
@@
 	(symbol
 		(lib_id "power:GND")
-		(at 203.2 106.68 0)
+		(at 180.34 104.14 0)
 		(unit 1)
 		(exclude_from_sim no)
@@
 		(fields_autoplaced yes)
 		(property "Reference" "#PWR0324"
-			(at 203.2 113.03 0)
+			(at 180.34 110.49 0)
 			(effects
 				(font
@@
 		)
 		(property "Value" "GND"
-			(at 203.2 111.1234 0)
+			(at 180.34 108.5834 0)
 			(effects
 				(font
@@
 		)
 		(property "Footprint" ""
-			(at 203.2 106.68 0)
+			(at 180.34 104.14 0)
 			(effects
 				(font
@@
 		)
 		(property "Datasheet" ""
-			(at 203.2 106.68 0)
+			(at 180.34 104.14 0)
 			(effects
 				(font
@@
 		)
 		(property "Description" ""
-			(at 203.2 106.68 0)
-			(effects
-				(font
+			(at 180.34 104.14 0)
+			(effects
+				(font

Commit message: added module connector
Parts:
- added J304: Conn_02x05_Top_Bottom, symbol Connector_Generic:Conn_02x05_Top_Bottom
Connections:
- net 3V3: now also J304.6 (Pin_6)
- net DR: now also J304.1 (Pin_1)
- net GND: now also J304.5 (Pin_5)
- net GP_CE: now also J304.2 (Pin_2)
- net INT: now also J304.4 (Pin_4)
- net MISO: now also J304.9 (Pin_9)
- net MOSI: now also J304.8 (Pin_8)
- net NCS: now also J304.7 (Pin_7)
- net SCL: now also J304.3 (Pin_3)
- net SCLK: now also J304.10 (Pin_10)

Commit message: Schematic 02 done
Parts:
- J302: footprint (none) -> Connector_PinHeader_2.54mm:PinHeader_1x02_P2.54mm_Vertical
- J304: footprint (none) -> Component_lib:PMK_Side_Conn_F
Changed lines of the file:
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@@
 			)
 		)
-		(property "Footprint" ""
+		(property "Footprint" "Component_lib:PMK_Side_Conn_F"
 			(at 182.88 88.9 0)
 			(effects
@@
 			)
 		)
-		(property "Footprint" ""
+		(property "Footprint" "Connector_PinHeader_2.54mm:PinHeader_1x02_P2.54mm_Vertical"
 			(at 43.18 114.3 0)
 			(effects

Commit message: routing ongoing
Parts:
- removed J304: Conn_02x05_Top_Bottom, Component_lib:PMK_Side_Conn_F, symbol Connector_Generic:Conn_02x05_Top_Bottom
- added J304: FH12-12S-0.5SH_55_, Component_lib:FH12-12S-0.5SH_55_, symbol Component_lib:FH12-12S-0.5SH_55_
Connections:
- net 3V3: now also J304.12
- net DR: now also J304.4
- net GND: now also J304.11
- net GP_CE: now also J304.3
- net MISO: now also J304.2
- net MOSI: now also J304.5
- net SCL: now also J304.9
- net SCLK: now also J304.1
- new net GPIO1: J304.6
- new net GPIO2: J304.7
- new net GPIO3: J304.8
- new net SDA: J304.10

Commit message: PMK_Keyboard_02 is done
Parts:
- removed J304: FH12-12S-0.5SH_55_, Component_lib:FH12-12S-0.5SH_55_, symbol Component_lib:FH12-12S-0.5SH_55_
- added J304, J305: FFC2B28-12-G, Component_lib:GCT_FFC2B28-12-G, symbol Component_lib:FFC2B28-12-G
Connections:
- net 3V3: now also J304.12, J305.12
- net DR: now also J304.4, J305.4
- net GND: now also J304.11, J304.S1 (SHIELD), J304.S2 (SHIELD), J305.11, J305.S1 (SHIELD), J305.S2 (SHIELD)
- net GPIO1: now also J304.6, J305.6
- net GPIO2: now also J304.7, J305.7
- net GPIO3: now also J304.8, J305.8
- net GP_CE: now also J304.3, J305.3
- net MISO: now also J304.2, J305.2
- net MOSI: now also J304.5, J305.5
- net SCL: now also J304.9, J305.9
- net SCLK: now also J304.1, J305.1
- net SDA: now also J304.10, J305.10
