File: Hardware/PMK_SpaceMouse/PMK_SpaceMouse_00/PMK_SpaceMouse_00.kicad_pcb (KiCad board)
At the start: 2 copper layers, 60.8 x 61.3 mm, 37 parts, among them J1 FFC2B28-12-G, U1 LDC1614, U2 LDC1612, X1 ASV-40.000MHz

Commit message: added production files for spacemouse_00
Parts:
- moved R2 0.70 mm to (123.2, 107.9)
- moved R3 0.10 mm to (135.2, 86.6)
- moved R4 0.10 mm to (137.1, 86.6)
Routing:
- net /3V3: track 21.0 -> 107.4 mm, vias 3 -> 7
- net /GPIO2: track 7.19 -> 50.2 mm, vias 1 -> 5
- net /GPIO1: track 9.36 -> 40.9 mm, vias 1 -> 3
- net GND: track 19.4 -> 27.2 mm, vias 1 -> 11
- net /40MHZ_CLK: track 39.5 -> 38.4 mm
- net Net-(U2-ADDR): track 2.18 -> 2.88 mm
