File: Hardware/PMK_SpaceMouse/PMK_SpaceMouse_01/PMK_SpaceMouse_01.kicad_sch (KiCad schematic)
At the start: 37 parts, among them J1 FFC2B28-12-G, U1 LDC1614, U2 LDC1612, X1 ASV-40.000MHz

Commit message: started pmk_03
Parts:
- added J2: vik-module-connector, vik:vik-module-connector-horizontal, symbol vik:vik-module-connector
Connections:
- net 3V3: now also J2.12 (3V3)
- net DR: now also J2.4 (GP_AD2)
- net GND: now also J2.11 (GND)
- net GPIO1: now also J2.6 (GP_AD1)
- net GPIO2: now also J2.7 (5V)
- net GPIO3: now also J2.8 (RGB_DO)
- net GP_CE: now also J2.3 (SPI_CS)
- net MISO: now also J2.2 (MISO)
- net MOSI: now also J2.5 (MOSI)
- net SCL: now also J2.9 (SCL)
- net SCLK: now also J2.1 (SCLK)
- net SDA: now also J2.10 (SDA)
