File: Hardware/PMK_Mouse/PMK_Mouse_00/PMK_Mouse_00.kicad_sch (KiCad schematic)
At the start: 2 parts, among them J1 PSoM_ESP32S2_Carrier_Board, U1 MP6543HGL-P

Commit message: started schematic
Parts:
- removed U1: MP6543HGL-P, Component_lib:QFN40P300X400X100-25N-D, symbol Component_lib:MP6543HGL-P
Other:
- added sheet Analog switch (Analog switch.kicad_sch)
- added sheet Haptic motor (Haptic motor.kicad_sch)
- added sheet Scroll wheel (Scroll wheel.kicad_sch)
- added sheet Sensor (Sensor.kicad_sch)
